Commit message: controller update

File: src/bopt_description/urdf/materials.xacro (robot description, xacro)
@@ -3,4 +3,7 @@
     <material name="black">
         <color rgba="0.1 0.1 0.1 1.0"/>
+    </material>
+    <material name="rubber_black">
+        <color rgba="0.05 0.05 0.05 1.0"/>
     </material>
     <material name="white">

File: src/bopt_description/urdf/robot.urdf.xacro (robot description, xacro)
@@ -76,5 +76,5 @@
                 <mesh filename="file:///home/jkw/bopt_ws/install/bopt_description/share/bopt_description/meshes/visual/drive_wheel.stl"/>
             </geometry>
-            <material name="black"/>
+            <material name="rubber_black"/>
         </visual>
         <collision>
@@ -177,5 +177,5 @@
                 <mesh filename="file:///home/jkw/bopt_ws/install/bopt_description/share/bopt_description/meshes/visual/casster_wheel.stl"/>
             </geometry>
-            <material name="black"/>
+            <material name="rubber_black"/>
         </visual>
         <collision>
@@ -207,5 +207,5 @@
                 <mesh filename="file:///home/jkw/bopt_ws/install/bopt_description/share/bopt_description/meshes/visual/casster_wheel.stl"/>
             </geometry>
-            <material name="black"/>
+            <material name="rubber_black"/>
         </visual>
         <collision>
@@ -408,6 +408,6 @@
         <origin xyz="0.477 0 -0.265" rpy="0 0 0"/>
         <axis xyz="0 0 1"/>
-        <limit lower="0" upper="0.095" effort="3000" velocity="0.05"/>
-        <dynamics damping="50" friction="10"/>
+        <limit lower="0" upper="0.095" effort="30000" velocity="0.05"/>
+        <dynamics damping="50" friction="20"/>
     </joint>
     <!-- ================================================================
@@ -499,5 +499,5 @@
                 <mesh filename="file:///home/jkw/bopt_ws/install/bopt_description/share/bopt_description/meshes/visual/front_wheel.stl"/>
             </geometry>
-            <material name="black"/>
+            <material name="rubber_black"/>
         </visual>
         <collision>
@@ -529,5 +529,5 @@
                 <mesh filename="file:///home/jkw/bopt_ws/install/bopt_description/share/bopt_description/meshes/visual/front_wheel.stl"/>
             </geometry>
-            <material name="black"/>
+            <material name="rubber_black"/>
         </visual>
         <collision>
@@ -610,23 +610,65 @@
          GAZEBO FRICTION PROPERTIES
          ================================================================ -->
+    <gazebo reference="front_lift_joint">
+      <kp>100000</kp>
+      <kd>1000</kd>
+    </gazebo>
     <gazebo reference="drive_wheel">
-        <mu1>2.0</mu1>
-        <mu2>2.0</mu2>
+        <mu1>1.2</mu1>
+        <mu2>1.2</mu2>
+        <kp>100000.0</kp>
+        <kd>100.0</kd>
+        <minDepth>0.001</minDepth>
+        <maxVel>0.1</maxVel>
+        <fdir1>1 0 0</fdir1>
     </gazebo>
     <gazebo reference="caster_wheel_left">
-        <mu1>1.0</mu1>
-        <mu2>1.0</mu2>
+        <mu1>0.8</mu1>   <!-- Forward friction -->
+        <mu2>0.02</mu2>  <!-- Sideways slip -->
+        <fdir1>1 0 0</fdir1>
+        <kp>100000.0</kp>
+        <kd>10.0</kd>
+        <minDepth>0.001</minDepth>
+        <maxVel>0.1</maxVel>
     </gazebo>
     <gazebo reference="caster_wheel_right">
-        <mu1>1.0</mu1>
-        <mu2>1.0</mu2>
+        <mu1>0.8</mu1>   <!-- Forward friction -->
+        <mu2>0.02</mu2>  <!-- Sideways slip -->
+        <fdir1>1 0 0</fdir1>
+        <kp>100000.0</kp>
+        <kd>10.0</kd>
+        <minDepth>0.001</minDepth>
+        <maxVel>0.1</maxVel>
     </gazebo>
     <gazebo reference="front_wheel_left">
         <mu1>1.0</mu1>
         <mu2>1.0</mu2>
+        <kp>100000.0</kp>
+        <kd>100.0</kd>
+        <minDepth>0.001</minDepth>
+        <maxVel>0.1</maxVel>
     </gazebo>
     <gazebo reference="front_wheel_right">
         <mu1>1.0</mu1>
         <mu2>1.0</mu2>
+        <kp>100000.0</kp>
+        <kd>100.0</kd>
+        <minDepth>0.001</minDepth>
+        <maxVel>0.1</maxVel>
+    </gazebo>
+    <gazebo reference="front_lift_joint">
+        <implicitSpringDamper>true</implicitSpringDamper>
+        <gravity>false</gravity>
+    </gazebo>
+    <!-- MIMIC STEERING JOINTS -->
+    <gazebo reference="front_wheel_shaft_left_joint">
+        <implicitSpringDamper>true</implicitSpringDamper>
+    </gazebo>
+    <gazebo reference="front_wheel_shaft_right_joint">
+        <implicitSpringDamper>true</implicitSpringDamper>
+    </gazebo>
+    <!-- DRIVE STEERING ASSEMBLY -->
+    <gazebo reference="drive_wheel_Ass_joint">
+        <implicitSpringDamper>true</implicitSpringDamper>
     </gazebo>
     <!--ROS2 Control Plugin-->
