Commit message: py controller

File: src/bopt_description/urdf/gazebo.xacro (robot description, xacro)
@@ -59,6 +59,6 @@
          ================================================================ -->
     <gazebo reference="drive_wheel">
-        <mu1>1.2</mu1>
-        <mu2>1.2</mu2>
+        <mu1>1.5</mu1>
+        <mu2>1.5</mu2>
         <kp>1000000.0</kp>
         <kd>100.0</kd>
@@ -68,6 +68,6 @@
     </gazebo>
     <gazebo reference="front_wheel_left">
-        <mu1>1.0</mu1>
-        <mu2>1.0</mu2>
+        <mu1>1.5</mu1>
+        <mu2>1.5</mu2>
         <kp>1000000.0</kp>
         <kd>100.0</kd>
@@ -76,6 +76,6 @@
     </gazebo>
     <gazebo reference="front_wheel_right">
-        <mu1>1.0</mu1>
-        <mu2>1.0</mu2>
+        <mu1>1.5</mu1>
+        <mu2>1.5</mu2>
         <kp>1000000.0</kp>
         <kd>100.0</kd>

File: src/bopt_description/urdf/robot.urdf.xacro (robot description, xacro)
@@ -87,6 +87,6 @@
                 <friction>
                     <ode>
-                        <mu>1.0</mu>
-                        <mu2>1.0</mu2>
+                        <mu>1.5</mu>
+                        <mu2>1.5</mu2>
                     </ode>
                 </friction>
@@ -180,10 +180,10 @@
             <material name="rubber_black"/>
         </visual>
-        <collision>
+        <!--<collision>
             <origin xyz="0 0 0" rpy="1.5708 0 0"/>
             <geometry>
                 <cylinder radius="0.050" length="0.055"/>
             </geometry>
-        </collision>
+        </collision>-->
         <inertial>
             <origin xyz="0 0 0" rpy="0 0 0"/>
@@ -210,10 +210,10 @@
             <material name="rubber_black"/>
         </visual>
-        <collision>
+        <!--<collision>
             <origin xyz="0 0 0" rpy="1.5708 0 0"/>
             <geometry>
                 <cylinder radius="0.050" length="0.055"/>
             </geometry>
-        </collision>
+        </collision>-->
         <inertial>
             <origin xyz="0 0 0" rpy="0 0 0"/>

Commit message: update controller

File: src/bopt_description/urdf/gazebo.xacro (robot description, xacro)
@@ -105,14 +105,30 @@
          ================================================================ -->
     <gazebo reference="front_lift_joint">
-        <implicitSpringDamper>true</implicitSpringDamper>
+        <physics>
+            <ode>
+                <implicit_spring_damper>true</implicit_spring_damper>
+            </ode>
+        </physics>
+    </gazebo>
+    <gazebo reference="front_wheel_shaft_right_joint">
+        <physics>
+            <ode>
+                <implicit_spring_damper>true</implicit_spring_damper>
+            </ode>
+        </physics>
     </gazebo>
     <gazebo reference="front_wheel_shaft_left_joint">
-        <implicitSpringDamper>true</implicitSpringDamper>
-    </gazebo>
-    <gazebo reference="front_wheel_shaft_right_joint">
-        <implicitSpringDamper>true</implicitSpringDamper>
+        <physics>
+            <ode>
+                <implicit_spring_damper>true</implicit_spring_damper>
+            </ode>
+        </physics>
     </gazebo>
     <gazebo reference="drive_wheel_Ass_joint">
-        <implicitSpringDamper>true</implicitSpringDamper>
+        <physics>
+            <ode>
+                <implicit_spring_damper>true</implicit_spring_damper>
+            </ode>
+        </physics>
     </gazebo>
     <!-- ================================================================

File: src/bopt_description/urdf/robot.urdf.xacro (robot description, xacro)
@@ -25,5 +25,5 @@
         <inertial>
             <origin xyz="0 0 -0.2500" rpy="0 0 0"/>
-            <mass value="80.0"/>
+            <mass value="200.0"/>
             <inertia ixx="3.46" ixy="0.0" ixz="0.0"
                      iyy="7.73" iyz="0.0"
@@ -398,5 +398,5 @@
         <inertial>
             <origin xyz="0.177 0 0" rpy="0 0 0"/>
-            <mass value="25"/>
+            <mass value="125"/>
             <inertia ixx="1.0" ixy="0.0" ixz="0.0"
                      iyy="2.0" iyz="0.0"
@@ -410,5 +410,5 @@
         <axis xyz="0 0 1"/>
         <limit lower="0" upper="0.095" effort="30000" velocity="0.05"/>
-        <dynamics damping="50" friction="20"/>
+        <dynamics damping="125" friction="15"/>
     </joint>
     <!-- ================================================================
@@ -446,8 +446,8 @@
         <limit lower="0"
             upper="0.785"
-            effort="5000"
-            velocity="2"/>  s
-        <dynamics damping="1.0"
-                friction="0.1"/>
+            effort="500000"
+            velocity="1"/>
+        <dynamics damping="80.0"
+                friction="0.8"/>
         <mimic joint="front_lift_joint"
                multiplier="7.725"
@@ -485,8 +485,8 @@
         <limit lower="0"
             upper="0.785"
-            effort="5000"
-            velocity="2"/>
-        <dynamics damping="1.0"
-                friction="0.1"/>
+            effort="500000"
+            velocity="1"/>
+        <dynamics damping="80.0"
+                friction="0.8"/>
         <mimic joint="front_lift_joint"
             multiplier="7.725"

Commit message: all things

File: src/bopt_description/urdf/gazebo.xacro (robot description, xacro)
@@ -135,4 +135,56 @@
          GAZEBO SENSOR PLUGINS
          ================================================================ -->
+    <!--imu link gazebo model-->
+    <gazebo reference="imu_link">
+      <sensor name="imu" type="imu">
+          <always_on>true</always_on>
+          <update_rate>100</update_rate>
+          <gz_frame_id>imu_link</gz_frame_id>
+          <visualize>true</visualize>
+          <topic>imu</topic>
+          <imu>
+            <angular_velocity>
+              <x>
+                <noise type="gaussian">
+                  <mean>0.0</mean>
+                  <stddev>2e-4</stddev>
+                </noise>
+              </x>
+              <y>
+                <noise type="gaussian">
+                  <mean>0.0</mean>
+                  <stddev>2e-4</stddev>
+                </noise>
+              </y>
+              <z>
+                <noise type="gaussian">
+                  <mean>0.0</mean>
+                  <stddev>2e-4</stddev>
+                </noise>
+              </z>
+            </angular_velocity>
+            <linear_acceleration>
+              <x>
+                <noise type="gaussian">
+                  <mean>0.0</mean>
+                  <stddev>1.7e-2</stddev>
+                </noise>
+              </x>
+              <y>
+                <noise type="gaussian">
+                  <mean>0.0</mean>
+                  <stddev>1.7e-2</stddev>
+                </noise>
+              </y>
+              <z>
+                <noise type="gaussian">
+                  <mean>0.0</mean>
+                  <stddev>1.7e-2</stddev>
+                </noise>
+              </z>
+            </linear_acceleration>
+          </imu>
+      </sensor>
+    </gazebo>
     <!-- 1. Front Top 2D LiDAR -->
     <gazebo reference="toplidar_front">
@@ -146,8 +198,8 @@
                 <scan>
                     <horizontal>
-                        <samples>360</samples>
-                        <resolution>1.0</resolution>
-                        <min_angle>-3.14159</min_angle>
-                        <max_angle>3.14159</max_angle>
+                        <samples>450</samples>
+                        <resolution>1.0</resolution>
+                        <min_angle>-1.570796</min_angle>
+                        <max_angle>1.570796</max_angle>
                     </horizontal>
                 </scan>
@@ -176,8 +228,8 @@
                 <scan>
                     <horizontal>
-                        <samples>360</samples>
-                        <resolution>1.0</resolution>
-                        <min_angle>-3.14159</min_angle>
-                        <max_angle>3.14159</max_angle>
+                        <samples>450</samples>
+                        <resolution>1.0</resolution>
+                        <min_angle>1.570796</min_angle>
+                        <max_angle>4.712389</max_angle>
                     </horizontal>
                 </scan>
@@ -206,8 +258,8 @@
                 <scan>
                     <horizontal>
-                        <samples>180</samples>
-                        <resolution>1.0</resolution>
-                        <min_angle>-1.5708</min_angle> <!-- 90 degree sweep -->
-                        <max_angle>1.5708</max_angle>
+                        <samples>450</samples>
+                        <resolution>1.0</resolution>
+                        <min_angle>-3.92699</min_angle>
+                        <max_angle>0.0</max_angle>
                     </horizontal>
                 </scan>
@@ -236,8 +288,8 @@
                 <scan>
                     <horizontal>
-                        <samples>180</samples>
-                        <resolution>1.0</resolution>
-                        <min_angle>-1.5708</min_angle> <!-- 90 degree sweep -->
-                        <max_angle>1.5708</max_angle>
+                        <samples>450</samples>
+                        <resolution>1.0</resolution>
+                        <min_angle>0.0</min_angle>
+                        <max_angle>3.92699</max_angle>
                     </horizontal>
                 </scan>
@@ -285,4 +337,63 @@
         </sensor>
     </gazebo>
+    <!--front safety lidar-->
+    <gazebo reference="front_lidar_frame_right">
+        <sensor name="front_right_lidar" type="gpu_lidar">
+            <always_on>true</always_on>
+            <update_rate>10.0</update_rate>
+            <visualize>true</visualize>
+            <topic>/lidar/front/right/scan</topic>
+            <gz_frame_id>front_lidar_frame_right</gz_frame_id>
+            <lidar>
+                <scan>
+                    <horizontal>
+                        <samples>450</samples>
+                        <resolution>1.0</resolution>
+                        <min_angle>-0.785398</min_angle>
+                        <max_angle>0.785398</max_angle>
+                    </horizontal>
+                </scan>
+                <range>
+                    <min>0.12</min>
+                    <max>10.0</max>
+                    <resolution>0.01</resolution>
+                </range>
+                <noise>
+                    <type>gaussian</type>
+                    <mean>0.0</mean>
+                    <stddev>0.01</stddev>
+                </noise>
+            </lidar>
+        </sensor>
+    </gazebo>
+    <gazebo reference="front_lidar_frame_left">
+        <sensor name="front_left_lidar" type="gpu_lidar">
+            <always_on>true</always_on>
+            <update_rate>10.0</update_rate>
+            <visualize>true</visualize>
+            <topic>/lidar/front/left/scan</topic>
+            <gz_frame_id>front_lidar_frame_left</gz_frame_id>
+            <lidar>
+                <scan>
+                    <horizontal>
+                        <samples>450</samples>
+                        <resolution>1.0</resolution>
+                        <min_angle>-0.785398</min_angle>
+                        <max_angle>0.785398</max_angle>
+                    </horizontal>
+                </scan>
+                <range>
+                    <min>0.12</min>
+                    <max>10.0</max>
+                    <resolution>0.01</resolution>
+                </range>
+                <noise>
+                    <type>gaussian</type>
+                    <mean>0.0</mean>
+                    <stddev>0.01</stddev>
+                </noise>
+            </lidar>
+        </sensor>
+    </gazebo>
     <!-- ================================================================
          ROS 2 CONTROL PLUGIN

File: src/bopt_description/urdf/robot.urdf.xacro (robot description, xacro)
@@ -69,4 +69,18 @@
         <limit lower="-3.14159" upper="3.14159" effort="1000" velocity="2"/>
         <dynamics damping="6" friction="0.1"/>
+    </joint>
+    <!--imu link -->
+    <link name="imu_link">
+        <inertial>
+            <origin xyz="0.0 0.0 0.0"/>
+            <mass value="0.01"/>
+            <inertia ixx="0.02" iyy="0.02" izz="0.02"
+                    ixy="0" ixz="0" iyz="0"/>
+        </inertial>
+    </link>
+    <joint name="imu_joint" type="fixed">
+        <parent link="drive_wheel_Ass"/>
+        <child link="imu_link"/>
+        <origin xyz="0 0 0.01"/>
     </joint>
     <!-- Drive wheel -->
@@ -180,10 +194,10 @@
             <material name="rubber_black"/>
         </visual>
-        <!--<collision>
+        <collision>
             <origin xyz="0 0 0" rpy="1.5708 0 0"/>
             <geometry>
                 <cylinder radius="0.050" length="0.055"/>
             </geometry>
-        </collision>-->
+        </collision>
         <inertial>
             <origin xyz="0 0 0" rpy="0 0 0"/>
@@ -210,10 +224,10 @@
             <material name="rubber_black"/>
         </visual>
-        <!--<collision>
+        <collision>
             <origin xyz="0 0 0" rpy="1.5708 0 0"/>
             <geometry>
                 <cylinder radius="0.050" length="0.055"/>
             </geometry>
-        </collision>-->
+        </collision>
         <inertial>
             <origin xyz="0 0 0" rpy="0 0 0"/>
@@ -377,5 +391,56 @@
         <parent link="base_link"/>
         <child link="top3dl_link"/>
-        <origin xyz="0.2556 0.0024 1.9831" rpy="0 0 0"/>
+        <origin xyz="0.2356 0.00 2.0731" rpy="0 0 0"/>
+    </joint>
+    <!--front safety lidar-->
+    <link name="front_lidar_frame_left">
+        <visual>
+            <origin xyz="0 0 0" rpy="0 0 -1.5708"/>
+            <geometry>
+                <mesh filename="file:///home/jkw/bopt_ws/install/bopt_description/share/bopt_description/meshes/visual/lidar19.stl"/>
+            </geometry>
+            <material name="gray"/>
+        </visual>
+        <collision>
+            <origin xyz="0 0 0" rpy="0 0 0"/>
+            <geometry>
+                <box size="0.05 0.05 0.05"/>
+            </geometry>
+        </collision>
+        <inertial>
+            <origin xyz="0 0 0" rpy="0 0 0"/>
+            <mass value="0.5"/>
+            <inertia ixx="0.001" ixy="0.0" ixz="0.0" iyy="0.001" iyz="0.0" izz="0.001"/>
+        </inertial>
+    </link>
+    <joint name="front_lidar_frame_left_joint" type="fixed">
+        <parent link="front_lift_link"/>
+        <child link="front_lidar_frame_left"/>
+        <origin xyz="1.233 0.180 0.025" rpy="3.14 0 0"/>
+    </joint>
+    <link name="front_lidar_frame_right">
+        <visual>
+            <origin xyz="0 0 0" rpy="0 0 -1.5708"/>
+            <geometry>
+                <mesh filename="file:///home/jkw/bopt_ws/install/bopt_description/share/bopt_description/meshes/visual/lidar19.stl"/>
+            </geometry>
+            <material name="gray"/>
+        </visual>
+        <collision>
+            <origin xyz="0 0 0" rpy="0 0 0"/>
+            <geometry>
+                <box size="0.05 0.05 0.05"/>
+            </geometry>
+        </collision>
+        <inertial>
+            <origin xyz="0 0 0" rpy="0 0 0"/>
+            <mass value="0.5"/>
+            <inertia ixx="0.001" ixy="0.0" ixz="0.0" iyy="0.001" iyz="0.0" izz="0.001"/>
+        </inertial>
+    </link>
+    <joint name="front_lidar_frame_right_joint" type="fixed">
+        <parent link="front_lift_link"/>
+        <child link="front_lidar_frame_right"/>
+        <origin xyz="1.233 -0.190 0.025" rpy="3.14 0 0"/>
     </joint>
     <!-- ================================================================

Commit message: multi

File: src/bopt_description/urdf/gazebo.xacro (robot description, xacro)
@@ -1,4 +1,6 @@
 <?xml version="1.0"?>
 <robot xmlns:xacro="http://www.ros.org/wiki/xacro">
+    <xacro:arg name="robot_namespace" default=""/>
+    <xacro:arg name="robot_param_node" default="robot_state_publisher"/>
     <!-- ================================================================
          GAZEBO MATERIALS
@@ -400,8 +402,14 @@
          ================================================================ -->
     <gazebo>
-        <plugin name="ign_ros2_control::IgnitionROS2ControlPlugin" filename="ign_ros2_control-system">
+        <plugin name="ign_ros2_control::IgnitionROS2ControlPlugin"
+                filename="ign_ros2_control-system">
             <robot_param>robot_description</robot_param>
             <robot_param_node>robot_state_publisher</robot_param_node>
-            <parameters>$(find bopt_description)/config/controller.yaml</parameters>
+            <parameters>
+                $(find bopt_description)/config/controller.yaml
+            </parameters>
+            <ros>
+                <namespace>$(arg robot_name)</namespace>
+            </ros>
         </plugin>
     </gazebo>

File: src/bopt_description/urdf/robot.urdf.xacro (robot description, xacro)
@@ -1,4 +1,7 @@
 <?xml version="1.0"?>
 <robot xmlns:xacro="http://www.ros.org/wiki/xacro" name="bopt_robot">
+    <xacro:arg name="robot_name" default=""/>
+    <xacro:arg name="robot_param_node" default="robot_state_publisher"/>
+    <xacro:property name="robot_name" value="$(arg robot_name)"/>
     <xacro:include filename="materials.xacro"/>
     <xacro:include filename="ros2_control.xacro"/>
@@ -618,4 +621,4 @@
         <dynamics damping="10" friction="6"/>
     </joint>
-    <xacro:ros2_control/>
+    <xacro:ros2_control robot_name="$(arg robot_name)"/>
 </robot>

File: src/bopt_description/urdf/ros2_control.xacro (robot description, xacro)
@@ -1,6 +1,6 @@
 <?xml version="1.0"?>
 <robot xmlns:xacro="http://www.ros.org/wiki/xacro">
-    <xacro:macro name="ros2_control">
-        <ros2_control name="my_robot_gazebo" type="system">
+    <xacro:macro name="ros2_control" params="robot_name">
+        <ros2_control name="${robot_name}_gazebo" type="system">
             <hardware>
                 <plugin>ign_ros2_control/IgnitionSystem</plugin>
