Commit message: ppts update and depth camer

File: src/bopt_description/urdf/gazebo.xacro (robot description, xacro)
@@ -137,4 +137,66 @@
          GAZEBO SENSOR PLUGINS
          ================================================================ -->
+    <!-- Ultrasonic sensor left -->
+    <gazebo reference="ultrasonic_link_left">
+        <sensor name="ultrasonic_sensor_left" type="gpu_lidar">
+            <always_on>true</always_on>
+            <visualize>true</visualize>
+            <update_rate>5</update_rate>
+            <topic>$(arg robot_namespace)/ultrasonic/left/range</topic>
+            <gz_frame_id>ultrasonic_link_left</gz_frame_id>
+            <lidar>
+                <scan>
+                    <horizontal>
+                        <samples>5</samples>
+                        <resolution>1</resolution>
+                        <min_angle>-0.1</min_angle>
+                        <max_angle>0.1</max_angle>
+                    </horizontal>
+                    <vertical>
+                        <samples>5</samples>
+                        <resolution>1</resolution>
+                        <min_angle>-0.1</min_angle>
+                        <max_angle>0.1</max_angle>
+                    </vertical>
+                </scan>
+                <range>
+                    <min>0.02</min>
+                    <max>5.0</max>
+                    <resolution>0.01</resolution>
+                </range>
+            </lidar>
+        </sensor>
+    </gazebo>
+    <!-- Ultrasonic sensor right -->
+    <gazebo reference="ultrasonic_link_right">
+        <sensor name="ultrasonic_sensor_right" type="gpu_lidar">
+            <always_on>true</always_on>
+            <visualize>true</visualize>
+            <update_rate>5</update_rate>
+            <topic>$(arg robot_namespace)/ultrasonic/right/range</topic>
+            <gz_frame_id>ultrasonic_link_right</gz_frame_id>
+            <lidar>
+                <scan>
+                    <horizontal>
+                        <samples>5</samples>
+                        <resolution>1</resolution>
+                        <min_angle>-0.1</min_angle>
+                        <max_angle>0.1</max_angle>
+                    </horizontal>
+                    <vertical>
+                        <samples>5</samples>
+                        <resolution>1</resolution>
+                        <min_angle>-0.1</min_angle>
+                        <max_angle>0.1</max_angle>
+                    </vertical>
+                </scan>
+                <range>
+                    <min>0.02</min>
+                    <max>5.0</max>
+                    <resolution>0.01</resolution>
+                </range>
+            </lidar>
+        </sensor>
+    </gazebo>
     <!--imu link gazebo model-->
     <gazebo reference="imu_link">
@@ -219,12 +281,33 @@
         </sensor>
     </gazebo>
-    <!-- 2. Back Top 2D LiDAR -->
-    <gazebo reference="toplidar_back">
-        <sensor name="back_2d_lidar" type="gpu_lidar">
-            <always_on>true</always_on>
-            <update_rate>10.0</update_rate>
-            <visualize>true</visualize>
-            <topic>$(arg robot_namespace)/lidar/back/scan</topic>
-            <gz_frame_id>toplidar_back</gz_frame_id>
+    <!-- 2. Back Depth Camera (replaces back lidar) -->
+    <gazebo reference="depth_camera_back">
+        <sensor name="back_depth_camera" type="rgbd_camera">
+            <always_on>true</always_on>
+            <update_rate>10.0</update_rate>
+            <topic>$(arg robot_namespace)/camera/back</topic>
+            <gz_frame_id>depth_camera_back_optical</gz_frame_id>
+            <camera>
+                <horizontal_fov>1.047198</horizontal_fov>
+                <image>
+                    <width>640</width>
+                    <height>480</height>
+                    <format>R8G8B8</format>
+                </image>
+                <clip>
+                    <near>0.05</near>
+                    <far>10.0</far>
+                </clip>
+            </camera>
+        </sensor>
+    </gazebo>
+    <!-- 3. Bottom Left 2D LiDAR -->
+    <gazebo reference="LLt">
+        <sensor name="left_bottom_lidar" type="gpu_lidar">
+            <always_on>true</always_on>
+            <update_rate>10.0</update_rate>
+            <visualize>true</visualize>
+            <topic>$(arg robot_namespace)/lidar/left/scan</topic>
+            <gz_frame_id>LLt</gz_frame_id>
             <lidar>
                 <scan>
@@ -232,6 +315,6 @@
                         <samples>450</samples>
                         <resolution>1.0</resolution>
-                        <min_angle>1.570796</min_angle>
-                        <max_angle>4.712389</max_angle>
+                        <min_angle>-3.92699</min_angle>
+                        <max_angle>0.0</max_angle>
                     </horizontal>
                 </scan>
@@ -249,12 +332,12 @@
         </sensor>
     </gazebo>
-    <!-- 3. Bottom Left 2D LiDAR -->
-    <gazebo reference="LLt">
-        <sensor name="left_bottom_lidar" type="gpu_lidar">
-            <always_on>true</always_on>
-            <update_rate>10.0</update_rate>
-            <visualize>true</visualize>
-            <topic>$(arg robot_namespace)/lidar/left/scan</topic>
-            <gz_frame_id>LLt</gz_frame_id>
+    <!-- 4. Bottom Right 2D LiDAR -->
+    <gazebo reference="LRt">
+        <sensor name="right_bottom_lidar" type="gpu_lidar">
+            <always_on>true</always_on>
+            <update_rate>10.0</update_rate>
+            <visualize>true</visualize>
+            <topic>$(arg robot_namespace)/lidar/right/scan</topic>
+            <gz_frame_id>LRt</gz_frame_id>
             <lidar>
                 <scan>
@@ -262,6 +345,6 @@
                         <samples>450</samples>
                         <resolution>1.0</resolution>
-                        <min_angle>-3.92699</min_angle>
-                        <max_angle>0.0</max_angle>
+                        <min_angle>0.0</min_angle>
+                        <max_angle>3.92699</max_angle>
                     </horizontal>
                 </scan>
@@ -279,34 +362,4 @@
         </sensor>
     </gazebo>
-    <!-- 4. Bottom Right 2D LiDAR -->
-    <gazebo reference="LRt">
-        <sensor name="right_bottom_lidar" type="gpu_lidar">
-            <always_on>true</always_on>
-            <update_rate>10.0</update_rate>
-            <visualize>true</visualize>
-            <topic>$(arg robot_namespace)/lidar/right/scan</topic>
-            <gz_frame_id>LRt</gz_frame_id>
-            <lidar>
-                <scan>
-                    <horizontal>
-                        <samples>450</samples>
-                        <resolution>1.0</resolution>
-                        <min_angle>0.0</min_angle>
-                        <max_angle>3.92699</max_angle>
-                    </horizontal>
-                </scan>
-                <range>
-                    <min>0.12</min>
-                    <max>30.0</max>
-                    <resolution>0.01</resolution>
-                </range>
-                <noise>
-                    <type>gaussian</type>
-                    <mean>0.0</mean>
-                    <stddev>0.01</stddev>
-                </noise>
-            </lidar>
-        </sensor>
-    </gazebo>
     <!-- 5. Top 3D LiDAR -->
     <gazebo reference="top3dl_link">
@@ -315,5 +368,5 @@
             <visualize>true</visualize>
             <topic>$(arg robot_namespace)/lidar/top3dl/scan</topic>
-            <update_rate>20</update_rate>
+            <update_rate>10.0</update_rate>
             <gz_frame_id>$(arg lidar_frame)</gz_frame_id>
             <lidar>

File: src/bopt_description/urdf/robot.urdf.xacro (robot description, xacro)
@@ -313,5 +313,5 @@
          ================================================================ -->
     <!-- Top 2D lidar - back -->
-    <link name="toplidar_back">
+    <!-- <link name="toplidar_back">
         <visual>
             <origin xyz="0 0 -0.005" rpy="0 0 1.5708"/>
@@ -339,4 +339,46 @@
         <child link="toplidar_back"/>
         <origin xyz="0.175 -0.0063 1.720" rpy="0 -0.45 0"/>
+    </joint> -->
+    <!--Depth camera instead of back lidar -->
+    <link name="depth_camera_back">
+        <visual>
+            <origin xyz="0 0 0" rpy="0 0 0"/>
+            <geometry>
+                <box size="0.05 0.05 0.05"/>
+            </geometry>
+            <material name="gray"/>
+        </visual>
+        <collision>
+            <origin xyz="0 0 0" rpy="0 0 0"/>
+            <geometry>
+                <box size="0.01 0.01 0.01"/>
+            </geometry>
+        </collision>
+        <inertial>
+            <origin xyz="0 0 0" rpy="0 0 0"/>
+            <mass value="0.1"/>
+            <inertia
+                ixx="0.01"
+                ixy="0.0"
+                ixz="0.0"
+                iyy="0.01"
+                iyz="0.0"
+                izz="0.01"/>
+        </inertial>
+    </link>
+    <joint name="depth_camera_joint_back" type="fixed">
+        <parent link="base_link"/>
+        <child link="depth_camera_back"/>
+        <origin
+            xyz="0.145 -0.0063 1.730"
+            rpy="3.14159 2.61759 0"/>
+    </joint>
+    <link name="depth_camera_back_optical"/>
+    <joint name="depth_camera_optical_joint_back" type="fixed">
+        <parent link="depth_camera_back"/>
+        <child link="depth_camera_back_optical"/>
+        <origin
+            xyz="0 0 0"
+            rpy="-1.5708 0 -1.5708"/>
     </joint>
     <!-- Top 2D lidar - front -->
@@ -623,4 +665,39 @@
         <dynamics damping="10" friction="6"/>
     </joint>
+    <!-- ultrasonic sensor for base left and right -->
+    <link name="ultrasonic_link_left">
+        <visual>
+            <geometry>
+                <box size="0.02 0.05 0.02"/>
+            </geometry>
+        </visual>
+        <collision>
+            <geometry>
+                <box size="0.02 0.05 0.02"/>
+            </geometry>
+        </collision>
+    </link>
+    <joint name="ultrasonic_joint_left" type="fixed">
+        <parent link="base_link"/>
+        <child link="ultrasonic_link_left"/>
+        <origin xyz="0.250 0.3704 0.600" rpy="0 0.0872665 0.1872665"/>
+    </joint>
+    <link name="ultrasonic_link_right">
+        <visual>
+            <geometry>
+                <box size="0.02 0.05 0.02"/>
+            </geometry>
+        </visual>
+        <collision>
+            <geometry>
+                <box size="0.02 0.05 0.02"/>
+            </geometry>
+        </collision>
+    </link>
+    <joint name="ultrasonic_joint_right" type="fixed">
+        <parent link="base_link"/>
+        <child link="ultrasonic_link_right"/>
+        <origin xyz="0.250 -0.3704 0.600" rpy="0 0.0872665 -0.1872665"/>
+    </joint>
     <xacro:ros2_control robot_name="$(arg robot_name)"/>
 </robot>

Commit message: pallte detection

File: src/bopt_description/urdf/gazebo.xacro (robot description, xacro)
@@ -134,4 +134,9 @@
         </physics>
     </gazebo>
+    <gazebo reference="limit_switch_bar_joint">
+        <implicitSpringDamper>true</implicitSpringDamper>
+        <springStiffness>5.0</springStiffness>
+        <springReference>0.0</springReference>
+    </gazebo>
     <!-- ================================================================
          GAZEBO SENSOR PLUGINS
@@ -287,5 +292,5 @@
             <update_rate>10.0</update_rate>
             <topic>$(arg robot_namespace)/camera/back</topic>
-            <gz_frame_id>depth_camera_back_optical</gz_frame_id>
+            <gz_frame_id>depth_camera_back</gz_frame_id>
             <camera>
                 <horizontal_fov>1.047198</horizontal_fov>

File: src/bopt_description/urdf/robot.urdf.xacro (robot description, xacro)
@@ -700,4 +700,56 @@
         <origin xyz="0.250 -0.3704 0.600" rpy="0 0.0872665 -0.1872665"/>
     </joint>
+    <!--Limit switch-->
+    <link name="limit_switch_link">
+        <visual>
+            <geometry>
+                <mesh filename="file:///home/jkw/bopt_ws/install/bopt_description/share/bopt_description/meshes/visual/limitswitch_frame.stl" scale="0.85 0.85 0.85"/>
+            </geometry>
+            <material name="gray"/>
+        </visual>
+        <collision>
+            <geometry>
+                <mesh filename="file:///home/jkw/bopt_ws/install/bopt_description/share/bopt_description/meshes/visual/limitswitch_frame.stl" scale="0.85 0.85 0.85"/>
+            </geometry>
+        </collision>
+    </link>
+    <joint name="limit_switch_joint" type="fixed">
+        <parent link="front_lift_link"/>
+        <child link="limit_switch_link"/>
+        <origin xyz="0.158 0 0.180" rpy="0 0 0"/>
+    </joint>
+    <link name="limit_switch_bar">
+        <visual>
+            <geometry>
+                <mesh filename="file:///home/jkw/bopt_ws/install/bopt_description/share/bopt_description/meshes/visual/limitswitch_bar.stl" scale="0.85 0.85 0.85"/>
+            </geometry>
+            <material name="black"/>
+        </visual>
+        <collision>
+            <origin xyz="0 0 -0.12" rpy="0 0 0"/>
+            <geometry>
+                <box size="0.02 0.04 0.25"/>
+            </geometry>
+        </collision>
+        <inertial>
+            <origin xyz="0 0 0" rpy="0 0 0"/>
+            <mass value="0.1"/>
+            <inertia ixx="0.001" ixy="0.0" ixz="0.0" iyy="0.001" iyz="0.0" izz="0.001"/>
+        </inertial>
+    </link>
+    <joint name="limit_switch_bar_joint" type="revolute">
+        <parent link="limit_switch_link"/>
+        <child link="limit_switch_bar"/>
+        <origin xyz="0.040 0 0.09" rpy="0 -0.200 0"/>
+        <axis xyz="0 1 0"/>
+        <limit
+            lower="-0.15708"
+            upper="0.15708"
+            effort="2"
+            velocity="1.0"/>
+        <dynamics
+            damping="0.5"
+            friction="0.1"/>
+    </joint>
     <xacro:ros2_control robot_name="$(arg robot_name)"/>
 </robot>

File: src/bopt_description/urdf/ros2_control.xacro (robot description, xacro)
@@ -63,4 +63,8 @@
                 <state_interface name="velocity"/>
             </joint>
+            <joint name="limit_switch_bar_joint">
+                <state_interface name="position"/>
+                <state_interface name="velocity"/>
+            </joint>
         </ros2_control>
     </xacro:macro>

Commit message: multi robot and palat pick and drp, and ppts and nmpc,workflow node update

File: src/bopt_description/urdf/gazebo.xacro (robot description, xacro)
@@ -3,4 +3,5 @@
     <xacro:arg name="robot_namespace" default=""/>
     <xacro:arg name="robot_param_node" default="robot_state_publisher"/>
+    <xacro:property name="ns" value="$(arg robot_namespace)"/>
     <!-- ================================================================
          GAZEBO MATERIALS
@@ -149,5 +150,5 @@
             <update_rate>5</update_rate>
             <topic>$(arg robot_namespace)/ultrasonic/left/range</topic>
-            <gz_frame_id>ultrasonic_link_left</gz_frame_id>
+            <gz_frame_id>${ns + '/' if ns != '' else ''}ultrasonic_link_left</gz_frame_id>
             <lidar>
                 <scan>
@@ -180,5 +181,5 @@
             <update_rate>5</update_rate>
             <topic>$(arg robot_namespace)/ultrasonic/right/range</topic>
-            <gz_frame_id>ultrasonic_link_right</gz_frame_id>
+            <gz_frame_id>${ns + '/' if ns != '' else ''}ultrasonic_link_right</gz_frame_id>
             <lidar>
                 <scan>
@@ -209,5 +210,5 @@
           <always_on>true</always_on>
           <update_rate>100</update_rate>
-          <gz_frame_id>imu_link</gz_frame_id>
+          <gz_frame_id>${ns + '/' if ns != '' else ''}imu_link</gz_frame_id>
           <visualize>true</visualize>
           <topic>$(arg robot_namespace)/imu</topic>
@@ -263,5 +264,5 @@
             <visualize>true</visualize>
             <topic>$(arg robot_namespace)/lidar/front/scan</topic>
-            <gz_frame_id>toplidar_front</gz_frame_id>
+            <gz_frame_id>${ns + '/' if ns != '' else ''}toplidar_front</gz_frame_id>
             <lidar>
                 <scan>
@@ -292,5 +293,5 @@
             <update_rate>30.0</update_rate>
             <topic>$(arg robot_namespace)/camera/back</topic>
-            <gz_frame_id>depth_camera_back</gz_frame_id>
+            <gz_frame_id>${ns + '/' if ns != '' else ''}depth_camera_back</gz_frame_id>
             <camera>
                 <horizontal_fov>1.3700834628155487</horizontal_fov>
@@ -314,5 +315,5 @@
             <visualize>true</visualize>
             <topic>$(arg robot_namespace)/lidar/left/scan</topic>
-            <gz_frame_id>LLt</gz_frame_id>
+            <gz_frame_id>${ns + '/' if ns != '' else ''}LLt</gz_frame_id>
             <lidar>
                 <scan>
@@ -344,5 +345,5 @@
             <visualize>true</visualize>
             <topic>$(arg robot_namespace)/lidar/right/scan</topic>
-            <gz_frame_id>LRt</gz_frame_id>
+            <gz_frame_id>${ns + '/' if ns != '' else ''}LRt</gz_frame_id>
             <lidar>
                 <scan>
@@ -404,5 +405,5 @@
             <visualize>true</visualize>
             <topic>$(arg robot_namespace)/Lidar_RFT</topic>
-            <gz_frame_id>front_lidar_frame_right</gz_frame_id>
+            <gz_frame_id>${ns + '/' if ns != '' else ''}front_lidar_frame_right</gz_frame_id>
             <lidar>
                 <scan>
@@ -433,5 +434,5 @@
             <visualize>true</visualize>
             <topic>$(arg robot_namespace)/Lidar_LFT</topic>
-            <gz_frame_id>front_lidar_frame_left</gz_frame_id>
+            <gz_frame_id>${ns + '/' if ns != '' else ''}front_lidar_frame_left</gz_frame_id>
             <lidar>
                 <scan>
