Commit message: bopt model

File: src/bopt_description/urdf/robot.urdf.xacro (robot description, xacro)
@@ -2,5 +2,9 @@
 <robot xmlns:xacro="http://www.ros.org/wiki/xacro" name="bopt_robot">
     <xacro:include filename="materials.xacro"/>
+    <!-- ================================================================
+         BASE LINKS
+         ================================================================ -->
     <link name="base_footprint"/>
+    <!-- Base chassis link -->
     <link name="base_link">
         <visual>
@@ -12,16 +16,27 @@
         </visual>
         <collision>
-            <origin rpy="0 0 0" xyz="0 0 0"/>
-            <geometry>
-                <box size="0.3 0.3 0.1"/>
-            </geometry>
-        </collision>
-    </link>
-     <joint name="base_footprint_joint" type="fixed">
+            <origin xyz="0 0 0.5" rpy="0 0 0"/>
+            <geometry>
+                <box size="0.5 0.7 0.7"/>
+            </geometry>
+        </collision>
+        <inertial>
+            <!-- mass=20 kg, box 0.3 x 0.3 x 0.1 m -->
+            <origin xyz="0 0 0" rpy="0 0 0"/>
+            <mass value="20.0"/>
+            <inertia ixx="0.1917" ixy="0.0" ixz="0.0"
+                     iyy="0.1917" iyz="0.0"
+                     izz="0.3000"/>
+        </inertial>
+    </link>
+    <joint name="base_footprint_joint" type="fixed">
         <parent link="base_footprint"/>
         <child link="base_link"/>
         <origin xyz="-1.20 0 0.3088" rpy="0 0 0"/>
     </joint>
-   <!--drive wheel holding ass-->
+    <!-- ================================================================
+         DRIVE WHEEL ASSEMBLY (Steering + Drive)
+         ================================================================ -->
+    <!-- Drive wheel steering assembly -->
     <link name="drive_wheel_Ass">
         <visual>
@@ -33,9 +48,17 @@
         </visual>
         <collision>
-            <origin rpy="0 0 0" xyz="0 0 0"/>
-            <geometry>
-                <box size="0.3 0.3 0.1"/>
-            </geometry>
-        </collision>
+            <origin xyz="0 0 00" rpy="0 0 0"/>
+            <geometry>
+                <box size="0.1 0.1 0.1"/>
+            </geometry>
+        </collision>
+        <inertial>
+            <!-- mass=2 kg, box 0.3 x 0.3 x 0.1 m -->
+            <origin xyz="0 0 0" rpy="0 0 0"/>
+            <mass value="2.0"/>
+            <inertia ixx="0.0192" ixy="0.0" ixz="0.0"
+                     iyy="0.0192" iyz="0.0"
+                     izz="0.0300"/>
+        </inertial>
     </link>
     <joint name="drive_wheel_Ass_joint" type="revolute">
@@ -43,9 +66,10 @@
         <child link="drive_wheel_Ass"/>
         <origin xyz="0 0 0" rpy="0 0 0"/>
-         <axis xyz="0 0 1"/>
+        <axis xyz="0 0 1"/>
         <limit lower="-1.5708" upper="1.5708" effort="1" velocity="1"/>
     </joint>
+    <!-- Drive wheel -->
     <link name="drive_wheel">
-         <visual>
+        <visual>
             <origin xyz="0 0 0" rpy="0 0 0"/>
             <geometry>
@@ -55,9 +79,17 @@
         </visual>
         <collision>
-            <origin rpy="0 0 0" xyz="0 0 0"/>
-            <geometry>
-                <cylinder radius="0.05215" length="0.03"/>
-            </geometry>
-        </collision>
+            <origin xyz="0 0 0" rpy="1.5708 0 0"/>
+            <geometry>
+                <cylinder radius="0.12215" length="0.06"/>
+            </geometry>
+        </collision>
+        <inertial>
+            <!-- mass=1 kg, solid cylinder r=0.05215 m, l=0.03 m -->
+            <origin xyz="0 0 0" rpy="0 0 0"/>
+            <mass value="1.0"/>
+            <inertia ixx="0.000933" ixy="0.0" ixz="0.0"
+                     iyy="0.000933" iyz="0.0"
+                     izz="0.001360"/>
+        </inertial>
     </link>
     <joint name="drive_wheel_joint" type="revolute">
@@ -68,6 +100,8 @@
         <limit lower="-3.1416" upper="3.1416" effort="1" velocity="1"/>
     </joint>
-    <!--end of sterring wheel part -->
-    <!--caster wheel holding ass-->
+    <!-- ================================================================
+         CASTER WHEEL ASSEMBLIES
+         ================================================================ -->
+    <!-- Caster assembly - right -->
     <link name="caster_wheel_ass_right">
         <visual>
@@ -79,9 +113,17 @@
         </visual>
         <collision>
-            <origin rpy="0 0 0" xyz="0 0 0"/>
-            <geometry>
-                <box size="0.3 0.3 0.1"/>
-            </geometry>
-        </collision>
+            <origin xyz="0 0 0" rpy="0 0 0"/>
+            <geometry>
+                <box size="0.1 0.1 0.1"/>
+            </geometry>
+        </collision>
+        <inertial>
+            <!-- mass=1 kg, box 0.3 x 0.3 x 0.1 m -->
+            <origin xyz="0 0 0" rpy="0 0 0"/>
+            <mass value="1.0"/>
+            <inertia ixx="0.0096" ixy="0.0" ixz="0.0"
+                     iyy="0.0096" iyz="0.0"
+                     izz="0.0150"/>
+        </inertial>
     </link>
     <joint name="caster_wheel_ass_joint_right" type="revolute">
@@ -92,4 +134,5 @@
         <limit lower="-3.14" upper="3.14" effort="1" velocity="1"/>
     </joint>
+    <!-- Caster assembly - left -->
     <link name="caster_wheel_ass_left">
         <visual>
@@ -101,9 +144,17 @@
         </visual>
         <collision>
-            <origin rpy="0 0 0" xyz="0 0 0"/>
-            <geometry>
-                <box size="0.3 0.3 0.1"/>
-            </geometry>
-        </collision>
+            <origin xyz="0 0 0" rpy="0 0 0"/>
+            <geometry>
+                <box size="0.1 0.1 0.1"/>
+            </geometry>
+        </collision>
+        <inertial>
+            <!-- mass=1 kg, box 0.3 x 0.3 x 0.1 m -->
+            <origin xyz="0 0 0" rpy="0 0 0"/>
+            <mass value="1.0"/>
+            <inertia ixx="0.0096" ixy="0.0" ixz="0.0"
+                     iyy="0.0096" iyz="0.0"
+                     izz="0.0150"/>
+        </inertial>
     </link>
     <joint name="caster_wheel_ass_joint_left" type="revolute">
@@ -114,18 +165,27 @@
         <limit lower="-3.14" upper="3.14" effort="1" velocity="1"/>
     </joint>
-    <!--wheel joint fot caster right-->
+    <!-- Caster wheel - right -->
     <link name="caster_wheel_right">
         <visual>
-           <geometry>
+            <origin xyz="0 0 0" rpy="0 0 0"/>
+            <geometry>
                 <mesh filename="package://bopt_description/meshes/visual/casster_wheel.stl" scale="1 1 1"/>
-           </geometry>
-           <material name="black"/>
-        </visual>
-        <collision>
-            <origin rpy="0 0 0" xyz="0 0 0"/>
+            </geometry>
+            <material name="black"/>
+        </visual>
+        <collision>
+            <origin xyz="0 0 0" rpy="1.5708 0 0"/>
             <geometry>
                 <cylinder radius="0.05215" length="0.03"/>
             </geometry>
         </collision>
+        <inertial>
+            <!-- mass=0.5 kg, solid cylinder r=0.05215 m, l=0.03 m -->
+            <origin xyz="0 0 0" rpy="0 0 0"/>
+            <mass value="0.5"/>
+            <inertia ixx="0.000467" ixy="0.0" ixz="0.0"
+                     iyy="0.000467" iyz="0.0"
+                     izz="0.000680"/>
+        </inertial>
     </link>
     <joint name="caster_wheel_joint_right" type="revolute">
@@ -136,18 +196,27 @@
         <limit lower="-3.14" upper="3.14" effort="1" velocity="1"/>
     </joint>
-    <!--wheel segment for caster left-->
-     <link name="caster_wheel_left">
-        <visual>
-           <geometry>
+    <!-- Caster wheel - left -->
+    <link name="caster_wheel_left">
+        <visual>
+            <origin xyz="0 0 0" rpy="0 0 0"/>
+            <geometry>
                 <mesh filename="package://bopt_description/meshes/visual/casster_wheel.stl" scale="1 1 1"/>
-           </geometry>
-           <material name="black"/>
-        </visual>
-        <collision>
-            <origin rpy="0 0 0" xyz="0 0 0"/>
+            </geometry>
+            <material name="black"/>
+        </visual>
+        <collision>
+            <origin xyz="0 0 0" rpy="1.5708 0 0"/>
             <geometry>
                 <cylinder radius="0.05215" length="0.03"/>
             </geometry>
         </collision>
+        <inertial>
+            <!-- mass=0.5 kg, solid cylinder r=0.05215 m, l=0.03 m -->
+            <origin xyz="0 0 0" rpy="0 0 0"/>
+            <mass value="0.5"/>
+            <inertia ixx="0.000467" ixy="0.0" ixz="0.0"
+                     iyy="0.000467" iyz="0.0"
+                     izz="0.000680"/>
+        </inertial>
     </link>
     <joint name="caster_wheel_joint_left" type="revolute">
@@ -158,6 +227,8 @@
         <limit lower="-3.14" upper="3.14" effort="1" velocity="1"/>
     </joint>
-    <!--end of caster wheel joint segment-->
-    <!--back  lidar segment-->
+    <!-- ================================================================
+         BOTTOM LIDAR SENSORS (rear corners)
+         ================================================================ -->
+    <!-- Bottom lidar - left rear -->
     <link name="LLt">
         <visual>
@@ -169,9 +240,17 @@
         </visual>
         <collision>
-            <origin rpy="0 0 0" xyz="0 0 0"/>
-            <geometry>
-                <box size="0.1 0.1 0.1"/>
-            </geometry>
-        </collision>
+            <origin xyz="0 0 0" rpy="0 0 0"/>
+            <geometry>
+                <box size="0.05 0.05 0.05"/>
+            </geometry>
+        </collision>
+        <inertial>
+            <!-- mass=0.2 kg, box 0.1 x 0.1 x 0.1 m -->
+            <origin xyz="0 0 0" rpy="0 0 0"/>
+            <mass value="0.2"/>
+            <inertia ixx="0.000333" ixy="0.0" ixz="0.0"
+                     iyy="0.000333" iyz="0.0"
+                     izz="0.000333"/>
+        </inertial>
     </link>
     <joint name="LLt_joint" type="fixed">
@@ -180,4 +259,5 @@
         <origin xyz="-0.1854 0.3704 -0.230" rpy="3.14 0 0"/>
     </joint>
+    <!-- Bottom lidar - right rear -->
     <link name="LRt">
         <visual>
@@ -189,9 +269,17 @@
         </visual>
         <collision>
-            <origin rpy="0 0 0" xyz="0 0 0"/>
-            <geometry>
-                <box size="0.1 0.1 0.1"/>
-            </geometry>
-        </collision>
+            <origin xyz="0 0 0" rpy="0 0 0"/>
+            <geometry>
+                <box size="0.05 0.05 0.05"/>
+            </geometry>
+        </collision>
+        <inertial>
+            <!-- mass=0.2 kg, box 0.1 x 0.1 x 0.1 m -->
+            <origin xyz="0 0 0" rpy="0 0 0"/>
+            <mass value="0.2"/>
+            <inertia ixx="0.000333" ixy="0.0" ixz="0.0"
+                     iyy="0.000333" iyz="0.0"
+                     izz="0.000333"/>
+        </inertial>
     </link>
     <joint name="LRt_joint" type="fixed">
@@ -200,5 +288,8 @@
         <origin xyz="-0.1854 -0.3704 -0.230" rpy="3.14 0 0"/>
     </joint>
-    <!--top lidar segment-->
+    <!-- ================================================================
+         TOP 2D LIDAR SENSORS
+         ================================================================ -->
+    <!-- Top 2D lidar - back -->
     <link name="toplidar_back">
         <visual>
@@ -210,9 +301,17 @@
         </visual>
         <collision>
-            <origin rpy="0 0 0" xyz="0 0 0"/>
-            <geometry>
-                <box size="0.1 0.1 0.1"/>
-            </geometry>
-        </collision>
+            <origin xyz="0 0 0" rpy="0 0 0"/>
+            <geometry>
+                <box size="0.05 0.05 0.05"/>
+            </geometry>
+        </collision>
+        <inertial>
+            <!-- mass=0.2 kg, box 0.1 x 0.1 x 0.1 m -->
+            <origin xyz="0 0 0" rpy="0 0 0"/>
+            <mass value="0.2"/>
+            <inertia ixx="0.000333" ixy="0.0" ixz="0.0"
+                     iyy="0.000333" iyz="0.0"
+                     izz="0.000333"/>
+        </inertial>
     </link>
     <joint name="toplidar_joint_back" type="fixed">
@@ -221,4 +320,5 @@
         <origin xyz="0.175 -0.0063 1.720" rpy="0 -0.45 0"/>
     </joint>
+    <!-- Top 2D lidar - front -->
     <link name="toplidar_front">
         <visual>
@@ -230,9 +330,17 @@
         </visual>
         <collision>
-            <origin rpy="0 0 0" xyz="0 0 0"/>
-            <geometry>
-                <box size="0.1 0.1 0.1"/>
-            </geometry>
-        </collision>
+            <origin xyz="0 0 0" rpy="0 0 0"/>
+            <geometry>
+                <box size="0.05 0.05 0.05"/>
+            </geometry>
+        </collision>
+        <inertial>
+            <!-- mass=0.2 kg, box 0.1 x 0.1 x 0.1 m -->
+            <origin xyz="0 0 0" rpy="0 0 0"/>
+            <mass value="0.2"/>
+            <inertia ixx="0.000333" ixy="0.0" ixz="0.0"
+                     iyy="0.000333" iyz="0.0"
+                     izz="0.000333"/>
+        </inertial>
     </link>
     <joint name="toplidar_joint_front" type="fixed">
@@ -241,5 +349,7 @@
         <origin xyz="0.288 -0.0063 1.66" rpy="0 0.47 0"/>
     </joint>
-    <!--top 3d lidar-->
+    <!-- ================================================================
+         TOP 3D LIDAR
+         ================================================================ -->
     <link name="top3dl_link">
         <visual>
@@ -251,9 +361,17 @@
         </visual>
         <collision>
-            <origin rpy="0 0 0" xyz="0 0 0"/>
+            <origin xyz="0 0 0" rpy="0 0 0"/>
             <geometry>
                 <box size="0.1 0.1 0.1"/>
             </geometry>
         </collision>
+        <inertial>
+            <!-- mass=0.5 kg, box 0.1 x 0.1 x 0.1 m -->
+            <origin xyz="0 0 0" rpy="0 0 0"/>
+            <mass value="0.5"/>
+            <inertia ixx="0.000833" ixy="0.0" ixz="0.0"
+                     iyy="0.000833" iyz="0.0"
+                     izz="0.000833"/>
+        </inertial>
     </link>
     <joint name="top3dl_joint" type="fixed">
@@ -262,7 +380,10 @@
         <origin xyz="0.2356 0.0024 1.9831" rpy="0 0 0"/>
     </joint>
-    <!--front part segment -->
+    <!-- ================================================================
+         FRONT LIFT MECHANISM
+         ================================================================ -->
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
Commit message: bopt model update

File: src/bopt_description/urdf/robot.urdf.xacro (robot description, xacro)
@@ -478,3 +478,66 @@
         <limit lower="-3.14" upper="3.14" effort="1" velocity="1"/>
     </joint>
+    <!--front wheel shaft- left -->
+    <link name="front_wheel_shaft_left">
+        <visual>
+            <origin xyz="0 0 0" rpy="-1.57080 0 0"/>
+            <geometry>
+                <mesh filename="package://bopt_description/meshes/visual/front_wheel_shaft.stl" scale="1 1 1"/>
+            </geometry>
+            <material name="black"/>
+        </visual>
+        <collision>
+            <origin xyz="0 0 0" rpy="0 0 0"/>
+            <geometry>
+                <cylinder radius="0.0615" length="0.1"/>
+            </geometry>
+        </collision>
+        <inertial>
+            <!-- mass=3 kg, solid cylinder r=0.175 m, l=0.1 m -->
+            <origin xyz="0.148 0 0" rpy="0 0 0"/>
+            <mass value="0.5"/>
+            <inertia ixx="0.039844" ixy="0.0" ixz="0.0"
+                     iyy="0.039844" iyz="0.0"
+                     izz="0.045938"/>
+        </inertial>
+    </link>
+    <joint name="front_wheel_shaft_left_joint" type="revolute">
+        <parent link="front_lift_link"/>
+        <child link="front_wheel_shaft_left"/>
+        <origin xyz="0.9211 0.1055 -0.01758" rpy="0 0 0"/>
+        <axis xyz="0 1 0"/>
+        <limit lower="0" upper="0.577" effort="0.2" velocity="100"/>
+        <dynamics damping="0.01" friction="0.0"/>
+    </joint>
+    <link name="front_wheel_shaft_right">
+        <visual>
+            <origin xyz="0 0 0" rpy="1.5708 0 0"/>
+            <geometry>
+                <mesh filename="package://bopt_description/meshes/visual/front_wheel_shaft.stl" scale="1 1 1"/>
+            </geometry>
+            <material name="black"/>
+        </visual>
+        <collision>
+            <origin xyz="0 0 0" rpy="0 0 0"/>
+            <geometry>
+                <cylinder radius="0.0615" length="0.1"/>
+            </geometry>
+        </collision>
+        <inertial>
+            <!-- mass=3 kg, solid cylinder r=0.175 m, l=0.1 m -->
+            <origin xyz="0.148 0 0" rpy="0 0 0"/>
+            <mass value="0.5"/>
+            <inertia ixx="0.039844" ixy="0.0" ixz="0.0"
+                     iyy="0.039844" iyz="0.0"
+                     izz="0.045938"/>
+        </inertial>
+    </link>
+    <joint name="front_wheel_shaft_right_joint" type="revolute">
+        <parent link="front_lift_link"/>
+        <child link="front_wheel_shaft_right"/>
+        <origin xyz="0.9211 -0.1135 -0.01758" rpy="0 0 0"/>
+        <axis xyz="0 1 0"/>
+        <limit lower="0" upper="0.577" effort="0.2" velocity="100"/>
+        <dynamics damping="0.01" friction="0.0"/>
+    </joint>
 </robot>
