Commit message: bopt model update

File: src/bopt_description/urdf/robot.urdf.xacro (robot description, xacro)
@@ -416,4 +416,67 @@
          FRONT WHEELS
          ================================================================ -->
+    <!--front wheel shaft- left -->
+    <link name="front_wheel_shaft_left">
+        <visual>
+            <origin xyz="0 0 0" rpy="-1.57080 0 0"/>
+            <geometry>
+                <mesh filename="package://bopt_description/meshes/visual/front_wheel_shaft.stl" scale="1 1 1"/>
+            </geometry>
+            <material name="black"/>
+        </visual>
+        <collision>
+            <origin xyz="0 0 0" rpy="0 0 0"/>
+            <geometry>
+                <box size="0.16 0.05 0.05"/>
+            </geometry>
+        </collision>
+        <inertial>
+            <!-- mass=3 kg, solid cylinder r=0.175 m, l=0.1 m -->
+            <origin xyz="0.148 0 0" rpy="0 0 0"/>
+            <mass value="1"/>
+            <inertia ixx="0.039844" ixy="0.0" ixz="0.0"
+                     iyy="0.039844" iyz="0.0"
+                     izz="0.045938"/>
+        </inertial>
+    </link>
+    <joint name="front_wheel_shaft_left_joint" type="revolute">
+        <parent link="front_lift_link"/>
+        <child link="front_wheel_shaft_left"/>
+        <origin xyz="0.9211 0.1055 -0.01758" rpy="0 0 0"/>
+        <axis xyz="0 1 0"/>
+        <limit lower="0" upper="0.7854" effort="2" velocity="100"/>
+        <dynamics damping="0.01" friction="0.0"/>
+    </joint>
+    <link name="front_wheel_shaft_right">
+        <visual>
+            <origin xyz="0 0 0" rpy="1.5708 0 0"/>
+            <geometry>
+                <mesh filename="package://bopt_description/meshes/visual/front_wheel_shaft.stl" scale="1 1 1"/>
+            </geometry>
+            <material name="black"/>
+        </visual>
+        <collision>
+            <origin xyz="0 0 0" rpy="0 0 0"/>
+            <geometry>
+                <box size="0.16 0.05 0.05"/>
+            </geometry>
+        </collision>
+        <inertial>
+            <!-- mass=3 kg, solid cylinder r=0.175 m, l=0.1 m -->
+            <origin xyz="0.148 0 0" rpy="0 0 0"/>
+            <mass value="1"/>
+            <inertia ixx="0.039844" ixy="0.0" ixz="0.0"
+                     iyy="0.039844" iyz="0.0"
+                     izz="0.045938"/>
+        </inertial>
+    </link>
+    <joint name="front_wheel_shaft_right_joint" type="revolute">
+        <parent link="front_lift_link"/>
+        <child link="front_wheel_shaft_right"/>
+        <origin xyz="0.9211 -0.1135 -0.01758" rpy="0 0 0"/>
+        <axis xyz="0 1 0"/>
+        <limit lower="0" upper="0.7854" effort="2" velocity="100"/>
+        <dynamics damping="0.01" friction="0.0"/>
+    </joint>
     <!-- Front wheel - right -->
     <link name="front_wheel_right">
@@ -441,7 +504,7 @@
     </link>
     <joint name="front_wheel_right_joint" type="revolute">
-        <parent link="base_link"/>
+        <parent link="front_wheel_shaft_right"/>
         <child link="front_wheel_right"/>
-        <origin xyz="1.5471 -0.1775 -0.2847" rpy="0 0 0"/>
+        <origin xyz="0.1488 -0.067 -0.0013" rpy="0 0 0"/>
         <axis xyz="0 1 0"/>
         <limit lower="-3.14" upper="3.14" effort="1" velocity="1"/>
@@ -472,72 +535,9 @@
     </link>
     <joint name="front_wheel_left_joint" type="revolute">
-        <parent link="base_link"/>
+        <parent link="front_wheel_shaft_left"/>
         <child link="front_wheel_left"/>
-        <origin xyz="1.5471 0.1775 -0.2847" rpy="0 0 0"/>
+        <origin xyz="0.1488 0.077 -0.0013" rpy="0 0 0"/>
         <axis xyz="0 1 0"/>
         <limit lower="-3.14" upper="3.14" effort="1" velocity="1"/>
     </joint>
-    <!--front wheel shaft- left -->
-    <link name="front_wheel_shaft_left">
-        <visual>
-            <origin xyz="0 0 0" rpy="-1.57080 0 0"/>
-            <geometry>
-                <mesh filename="package://bopt_description/meshes/visual/front_wheel_shaft.stl" scale="1 1 1"/>
-            </geometry>
-            <material name="black"/>
-        </visual>
-        <collision>
-            <origin xyz="0 0 0" rpy="0 0 0"/>
-            <geometry>
-                <cylinder radius="0.0615" length="0.1"/>
-            </geometry>
-        </collision>
-        <inertial>
-            <!-- mass=3 kg, solid cylinder r=0.175 m, l=0.1 m -->
-            <origin xyz="0.148 0 0" rpy="0 0 0"/>
-            <mass value="0.5"/>
-            <inertia ixx="0.039844" ixy="0.0" ixz="0.0"
-                     iyy="0.039844" iyz="0.0"
-                     izz="0.045938"/>
-        </inertial>
-    </link>
-    <joint name="front_wheel_shaft_left_joint" type="revolute">
-        <parent link="front_lift_link"/>
-        <child link="front_wheel_shaft_left"/>
-        <origin xyz="0.9211 0.1055 -0.01758" rpy="0 0 0"/>
-        <axis xyz="0 1 0"/>
-        <limit lower="0" upper="0.577" effort="0.2" velocity="100"/>
-        <dynamics damping="0.01" friction="0.0"/>
-    </joint>
-    <link name="front_wheel_shaft_right">
-        <visual>
-            <origin xyz="0 0 0" rpy="1.5708 0 0"/>
-            <geometry>
-                <mesh filename="package://bopt_description/meshes/visual/front_wheel_shaft.stl" scale="1 1 1"/>
-            </geometry>
-            <material name="black"/>
-        </visual>
-        <collision>
-            <origin xyz="0 0 0" rpy="0 0 0"/>
-            <geometry>
-                <cylinder radius="0.0615" length="0.1"/>
-            </geometry>
-        </collision>
-        <inertial>
-            <!-- mass=3 kg, solid cylinder r=0.175 m, l=0.1 m -->
-            <origin xyz="0.148 0 0" rpy="0 0 0"/>
-            <mass value="0.5"/>
-            <inertia ixx="0.039844" ixy="0.0" ixz="0.0"
-                     iyy="0.039844" iyz="0.0"
-                     izz="0.045938"/>
-        </inertial>
-    </link>
-    <joint name="front_wheel_shaft_right_joint" type="revolute">
-        <parent link="front_lift_link"/>
-        <child link="front_wheel_shaft_right"/>
-        <origin xyz="0.9211 -0.1135 -0.01758" rpy="0 0 0"/>
-        <axis xyz="0 1 0"/>
-        <limit lower="0" upper="0.577" effort="0.2" velocity="100"/>
-        <dynamics damping="0.01" friction="0.0"/>
-    </joint>
 </robot>
