Commit message: add extra file and update urdf

File: src/bopt_description/urdf/robot.urdf.xacro (robot description, xacro)
@@ -11,21 +11,20 @@
             <origin xyz="0 0 0" rpy="0 0 0"/>
             <geometry>
-                <mesh filename="package://bopt_description/meshes/visual/Base.stl" scale="1 1 1"/>
+                <mesh filename="file:///home/jkw/bopt_ws/install/bopt_description/share/bopt_description/meshes/visual/Base.stl"/>
             </geometry>
             <material name="blue"/>
         </visual>
         <collision>
-            <origin xyz="0 0 0.5" rpy="0 0 0"/>
-            <geometry>
-                <box size="0.5 0.7 0.7"/>
-            </geometry>
-        </collision>
-        <inertial>
-            <!-- mass=20 kg, box 0.3 x 0.3 x 0.1 m -->
+            <origin xyz="0 0 0" rpy="0 0 0"/>
+            <geometry>
+                <mesh filename="file:///home/jkw/bopt_ws/install/bopt_description/share/bopt_description/meshes/visual/Base.stl"/>
+            </geometry>
+        </collision>
+        <inertial>
             <origin xyz="0 0 0" rpy="0 0 0"/>
             <mass value="20.0"/>
-            <inertia ixx="0.1917" ixy="0.0" ixz="0.0"
-                     iyy="0.1917" iyz="0.0"
-                     izz="0.3000"/>
+            <inertia ixx="0.01" ixy="0.0" ixz="0.0"
+                     iyy="0.01" iyz="0.0"
+                     izz="0.01"/>
         </inertial>
     </link>
@@ -33,5 +32,5 @@
         <parent link="base_footprint"/>
         <child link="base_link"/>
-        <origin xyz="-1.20 0 0.3088" rpy="0 0 0"/>
+        <origin xyz="-1.2 0 0.350" rpy="0 0 0"/>
     </joint>
     <!-- ================================================================
@@ -43,5 +42,5 @@
             <origin xyz="0 0 0" rpy="0 0 0"/>
             <geometry>
-                <mesh filename="package://bopt_description/meshes/visual/drive_wheel_ass.stl" scale="1 1 1"/>
+                <mesh filename="file:///home/jkw/bopt_ws/install/bopt_description/share/bopt_description/meshes/visual/drive_wheel_ass.stl"/>
             </geometry>
             <material name="yellow"/>
@@ -50,5 +49,5 @@
             <origin xyz="0 0 00" rpy="0 0 0"/>
             <geometry>
-                <box size="0.1 0.1 0.1"/>
+                <mesh filename="file:///home/jkw/bopt_ws/install/bopt_description/share/bopt_description/meshes/visual/drive_wheel_ass.stl"/>
             </geometry>
         </collision>
@@ -57,7 +56,7 @@
             <origin xyz="0 0 0" rpy="0 0 0"/>
             <mass value="2.0"/>
-            <inertia ixx="0.0192" ixy="0.0" ixz="0.0"
-                     iyy="0.0192" iyz="0.0"
-                     izz="0.0300"/>
+            <inertia ixx="0.01" ixy="0.0" ixz="0.0"
+                     iyy="0.01" iyz="0.0"
+                     izz="0.01"/>
         </inertial>
     </link>
@@ -68,4 +67,5 @@
         <axis xyz="0 0 1"/>
         <limit lower="-1.5708" upper="1.5708" effort="1" velocity="1"/>
+        <dynamics damping="0.1" friction="0.1"/>
     </joint>
     <!-- Drive wheel -->
@@ -74,12 +74,12 @@
             <origin xyz="0 0 0" rpy="0 0 0"/>
             <geometry>
-                <mesh filename="package://bopt_description/meshes/visual/drive_wheel.stl" scale="1 1 1"/>
-            </geometry>
-            <material name="black"/>
-        </visual>
-        <collision>
-            <origin xyz="0 0 0" rpy="1.5708 0 0"/>
-            <geometry>
-                <cylinder radius="0.12215" length="0.06"/>
+                <mesh filename="file:///home/jkw/bopt_ws/install/bopt_description/share/bopt_description/meshes/visual/drive_wheel.stl"/>
+            </geometry>
+            <material name="black"/>
+        </visual>
+        <collision>
+            <origin xyz="0 0 0" rpy="0 0 0"/>
+            <geometry>
+                <mesh filename="file:///home/jkw/bopt_ws/install/bopt_description/share/bopt_description/meshes/visual/drive_wheel.stl"/>
             </geometry>
         </collision>
@@ -88,15 +88,15 @@
             <origin xyz="0 0 0" rpy="0 0 0"/>
             <mass value="1.0"/>
-            <inertia ixx="0.000933" ixy="0.0" ixz="0.0"
-                     iyy="0.000933" iyz="0.0"
-                     izz="0.001360"/>
-        </inertial>
-    </link>
-    <joint name="drive_wheel_joint" type="revolute">
+            <inertia ixx="0.01" ixy="0.0" ixz="0.0"
+                     iyy="0.01" iyz="0.0"
+                     izz="0.01"/>
+        </inertial>
+    </link>
+    <joint name="drive_wheel_joint" type="continuous">
         <parent link="drive_wheel_Ass"/>
         <child link="drive_wheel"/>
-        <origin xyz="0 0 -0.2233" rpy="0 0 0"/>
-        <axis xyz="0 1 0"/>
-        <limit lower="-3.1416" upper="3.1416" effort="1" velocity="1"/>
+        <origin xyz="0 0 -0.222" rpy="0 0 0"/>
+        <axis xyz="0 1 0"/>
+        <dynamics damping="0.1" friction="0.1"/>
     </joint>
     <!-- ================================================================
@@ -108,5 +108,5 @@
             <origin xyz="0 0 0" rpy="0 0 0"/>
             <geometry>
-                <mesh filename="package://bopt_description/meshes/visual/caster_wheel_ass.stl" scale="1 1 1"/>
+                <mesh filename="file:///home/jkw/bopt_ws/install/bopt_description/share/bopt_description/meshes/visual/caster_wheel_ass.stl"/>
             </geometry>
             <material name="yellow"/>
@@ -115,5 +115,5 @@
             <origin xyz="0 0 0" rpy="0 0 0"/>
             <geometry>
-                <box size="0.1 0.1 0.1"/>
+                <mesh filename="file:///home/jkw/bopt_ws/install/bopt_description/share/bopt_description/meshes/visual/caster_wheel_ass.stl"/>
             </geometry>
         </collision>
@@ -122,15 +122,15 @@
             <origin xyz="0 0 0" rpy="0 0 0"/>
             <mass value="1.0"/>
-            <inertia ixx="0.0096" ixy="0.0" ixz="0.0"
-                     iyy="0.0096" iyz="0.0"
-                     izz="0.0150"/>
-        </inertial>
-    </link>
-    <joint name="caster_wheel_ass_joint_right" type="revolute">
+            <inertia ixx="0.01" ixy="0.0" ixz="0.0"
+                     iyy="0.01" iyz="0.0"
+                     izz="0.01"/>
+        </inertial>
+    </link>
+    <joint name="caster_wheel_ass_joint_right" type="continuous">
         <parent link="base_link"/>
         <child link="caster_wheel_ass_right"/>
         <origin xyz="0 -0.255 -0.20515" rpy="0 0 0"/>
         <axis xyz="0 0 1"/>
-        <limit lower="-3.14" upper="3.14" effort="1" velocity="1"/>
+        <dynamics damping="0.1" friction="0.1"/>
     </joint>
     <!-- Caster assembly - left -->
@@ -139,5 +139,5 @@
             <origin xyz="0 0 0" rpy="0 0 0"/>
             <geometry>
-                <mesh filename="package://bopt_description/meshes/visual/caster_wheel_ass.stl" scale="1 1 1"/>
+                <mesh filename="file:///home/jkw/bopt_ws/install/bopt_description/share/bopt_description/meshes/visual/caster_wheel_ass.stl"/>
             </geometry>
             <material name="yellow"/>
@@ -146,5 +146,5 @@
             <origin xyz="0 0 0" rpy="0 0 0"/>
             <geometry>
-                <box size="0.1 0.1 0.1"/>
+                <mesh filename="file:///home/jkw/bopt_ws/install/bopt_description/share/bopt_description/meshes/visual/caster_wheel_ass.stl"/>
             </geometry>
         </collision>
@@ -153,15 +153,15 @@
             <origin xyz="0 0 0" rpy="0 0 0"/>
             <mass value="1.0"/>
-            <inertia ixx="0.0096" ixy="0.0" ixz="0.0"
-                     iyy="0.0096" iyz="0.0"
-                     izz="0.0150"/>
-        </inertial>
-    </link>
-    <joint name="caster_wheel_ass_joint_left" type="revolute">
+            <inertia ixx="0.01" ixy="0.0" ixz="0.0"
+                     iyy="0.01" iyz="0.0"
+                     izz="0.01"/>
+        </inertial>
+    </link>
+    <joint name="caster_wheel_ass_joint_left" type="continuous">
         <parent link="base_link"/>
         <child link="caster_wheel_ass_left"/>
         <origin xyz="0 0.255 -0.20515" rpy="0 0 0"/>
         <axis xyz="0 0 1"/>
-        <limit lower="-3.14" upper="3.14" effort="1" velocity="1"/>
+        <dynamics damping="0.1" friction="0.1"/>
     </joint>
     <!-- Caster wheel - right -->
@@ -170,12 +170,12 @@
             <origin xyz="0 0 0" rpy="0 0 0"/>
             <geometry>
-                <mesh filename="package://bopt_description/meshes/visual/casster_wheel.stl" scale="1 1 1"/>
-            </geometry>
-            <material name="black"/>
-        </visual>
-        <collision>
-            <origin xyz="0 0 0" rpy="1.5708 0 0"/>
-            <geometry>
-                <cylinder radius="0.05215" length="0.03"/>
+                <mesh filename="file:///home/jkw/bopt_ws/install/bopt_description/share/bopt_description/meshes/visual/casster_wheel.stl"/>
+            </geometry>
+            <material name="black"/>
+        </visual>
+        <collision>
+            <origin xyz="0 0 0" rpy="0 0 0"/>
+            <geometry>
+                <mesh filename="file:///home/jkw/bopt_ws/install/bopt_description/share/bopt_description/meshes/visual/casster_wheel.stl"/>
             </geometry>
         </collision>
@@ -184,15 +184,15 @@
             <origin xyz="0 0 0" rpy="0 0 0"/>
             <mass value="0.5"/>
-            <inertia ixx="0.000467" ixy="0.0" ixz="0.0"
-                     iyy="0.000467" iyz="0.0"
-                     izz="0.000680"/>
-        </inertial>
-    </link>
-    <joint name="caster_wheel_joint_right" type="revolute">
+            <inertia ixx="0.01" ixy="0.0" ixz="0.0"
+                     iyy="0.01" iyz="0.0"
+                     izz="0.01"/>
+        </inertial>
+    </link>
+    <joint name="caster_wheel_joint_right" type="continuous">
         <parent link="caster_wheel_ass_right"/>
         <child link="caster_wheel_right"/>
-        <origin xyz="0 0 -0.080" rpy="0 0 0"/>
-        <axis xyz="0 1 0"/>
-        <limit lower="-3.14" upper="3.14" effort="1" velocity="1"/>
+        <origin xyz="0 0 -0.08105" rpy="0 0 0"/>
+        <axis xyz="0 1 0"/>
+        <dynamics damping="0.1" friction="0.1"/>
     </joint>
     <!-- Caster wheel - left -->
@@ -201,12 +201,12 @@
             <origin xyz="0 0 0" rpy="0 0 0"/>
             <geometry>
-                <mesh filename="package://bopt_description/meshes/visual/casster_wheel.stl" scale="1 1 1"/>
-            </geometry>
-            <material name="black"/>
-        </visual>
-        <collision>
-            <origin xyz="0 0 0" rpy="1.5708 0 0"/>
-            <geometry>
-                <cylinder radius="0.05215" length="0.03"/>
+                <mesh filename="file:///home/jkw/bopt_ws/install/bopt_description/share/bopt_description/meshes/visual/casster_wheel.stl"/>
+            </geometry>
+            <material name="black"/>
+        </visual>
+        <collision>
+            <origin xyz="0 0 0" rpy="0 0 0"/>
+            <geometry>
+                <mesh filename="file:///home/jkw/bopt_ws/install/bopt_description/share/bopt_description/meshes/visual/casster_wheel.stl"/>
             </geometry>
         </collision>
@@ -215,15 +215,15 @@
             <origin xyz="0 0 0" rpy="0 0 0"/>
             <mass value="0.5"/>
-            <inertia ixx="0.000467" ixy="0.0" ixz="0.0"
-                     iyy="0.000467" iyz="0.0"
-                     izz="0.000680"/>
-        </inertial>
-    </link>
-    <joint name="caster_wheel_joint_left" type="revolute">
+            <inertia ixx="0.01" ixy="0.0" ixz="0.0"
+                     iyy="0.01" iyz="0.0"
+                     izz="0.01"/>
+        </inertial>
+    </link>
+    <joint name="caster_wheel_joint_left" type="continuous">
         <parent link="caster_wheel_ass_left"/>
         <child link="caster_wheel_left"/>
-        <origin xyz="0 0 -0.080" rpy="0 0 0"/>
-        <axis xyz="0 1 0"/>
-        <limit lower="-3.14" upper="3.14" effort="1" velocity="1"/>
+        <origin xyz="0 0 -0.08105" rpy="0 0 0"/>
+        <axis xyz="0 1 0"/>
+        <dynamics damping="0.1" friction="0.1"/>
     </joint>
     <!-- ================================================================
@@ -235,5 +235,5 @@
             <origin xyz="0 0 -0.009" rpy="0 0 2.356"/>
             <geometry>
-                <mesh filename="package://bopt_description/meshes/visual/lidar19.stl" scale="1 1 1"/>
+                <mesh filename="file:///home/jkw/bopt_ws/install/bopt_description/share/bopt_description/meshes/visual/lidar19.stl"/>
             </geometry>
             <material name="gray"/>
@@ -249,7 +249,7 @@
             <origin xyz="0 0 0" rpy="0 0 0"/>
             <mass value="0.2"/>
-            <inertia ixx="0.000333" ixy="0.0" ixz="0.0"
-                     iyy="0.000333" iyz="0.0"
-                     izz="0.000333"/>
+            <inertia ixx="0.01" ixy="0.0" ixz="0.0"
+                     iyy="0.01" iyz="0.0"
+                     izz="0.01"/>
         </inertial>
     </link>
@@ -264,5 +264,5 @@
             <origin xyz="0 0 -0.009" rpy="0 0 0.784"/>
             <geometry>
-                <mesh filename="package://bopt_description/meshes/visual/lidar19.stl" scale="1 1 1"/>
+                <mesh filename="file:///home/jkw/bopt_ws/install/bopt_description/share/bopt_description/meshes/visual/lidar19.stl"/>
             </geometry>
             <material name="gray"/>
@@ -278,7 +278,7 @@
             <origin xyz="0 0 0" rpy="0 0 0"/>
             <mass value="0.2"/>
-            <inertia ixx="0.000333" ixy="0.0" ixz="0.0"
-                     iyy="0.000333" iyz="0.0"
-                     izz="0.000333"/>
+            <inertia ixx="0.01" ixy="0.0" ixz="0.0"
+                     iyy="0.01" iyz="0.0"
+                     izz="0.01"/>
         </inertial>
     </link>
@@ -296,5 +296,5 @@
             <origin xyz="0 0 -0.005" rpy="0 0 1.5708"/>
             <geometry>
-                <mesh filename="package://bopt_description/meshes/visual/lidar19.stl" scale="1 1 1"/>
+                <mesh filename="file:///home/jkw/bopt_ws/install/bopt_description/share/bopt_description/meshes/visual/lidar19.stl"/>
             </geometry>
             <material name="gray"/>
@@ -310,7 +310,7 @@
             <origin xyz="0 0 0" rpy="0 0 0"/>
             <mass value="0.2"/>
-            <inertia ixx="0.000333" ixy="0.0" ixz="0.0"
-                     iyy="0.000333" iyz="0.0"
-                     izz="0.000333"/>
+            <inertia ixx="0.01" ixy="0.0" ixz="0.0"
+                     iyy="0.01" iyz="0.0"
+                     izz="0.01"/>
         </inertial>
     </link>
@@ -325,5 +325,5 @@
             <origin xyz="0 0 -0.003" rpy="0 0 -1.5708"/>
             <geometry>
-                <mesh filename="package://bopt_description/meshes/visual/lidar19.stl" scale="1 1 1"/>
+                <mesh filename="file:///home/jkw/bopt_ws/install/bopt_description/share/bopt_description/meshes/visual/lidar19.stl"/>
             </geometry>
             <material name="gray"/>
@@ -339,7 +339,7 @@
             <origin xyz="0 0 0" rpy="0 0 0"/>
             <mass value="0.2"/>
-            <inertia ixx="0.000333" ixy="0.0" ixz="0.0"
-                     iyy="0.000333" iyz="0.0"
-                     izz="0.000333"/>
+            <inertia ixx="0.01" ixy="0.0" ixz="0.0"
+                     iyy="0.01" iyz="0.0"
+                     izz="0.01"/>
         </inertial>
     </link>
@@ -356,5 +356,5 @@
             <origin xyz="0 0 0" rpy="0 0 0"/>
             <geometry>
-                <mesh filename="package://bopt_description/meshes/visual/3Dlidar.stl" scale="1 1 1"/>
+                <mesh filename="file:///home/jkw/bopt_ws/install/bopt_description/share/bopt_description/meshes/visual/3Dlidar.stl"/>
             </geometry>
             <material name="gray"/>
@@ -370,7 +370,7 @@
             <origin xyz="0 0 0" rpy="0 0 0"/>
             <mass value="0.5"/>
-            <inertia ixx="0.000833" ixy="0.0" ixz="0.0"
-                     iyy="0.000833" iyz="0.0"
-                     izz="0.000833"/>
+            <inertia ixx="0.01" ixy="0.0" ixz="0.0"
+                     iyy="0.01" iyz="0.0"
+                     izz="0.01"/>
         </inertial>
     </link>
@@ -387,5 +387,5 @@
             <origin xyz="0 0 0" rpy="0 0 0"/>
             <geometry>
-                <mesh filename="package://bopt_description/meshes/visual/front.stl" scale="1 1 1"/>
+                <mesh filename="file:///home/jkw/bopt_ws/install/bopt_description/share/bopt_description/meshes/visual/front.stl"/>
             </geometry>
             <material name="black"/>
@@ -394,5 +394,5 @@
             <origin xyz="0.22 0 0.1" rpy="0 0 0"/>
             <geometry>
-                <box size="0.8 0.7 0.2"/>
+                <box size="0.5 0.6 0.1"/>
             </geometry>
         </collision>
@@ -401,7 +401,7 @@
             <origin xyz="0 0 0" rpy="0 0 0"/>
             <mass value="3.0"/>
-            <inertia ixx="0.005000" ixy="0.0" ixz="0.0"
-                     iyy="0.005000" iyz="0.0"
-                     izz="0.005000"/>
+            <inertia ixx="0.01" ixy="0.0" ixz="0.0"
+                     iyy="0.01" iyz="0.0"
+                     izz="0.01"/>
         </inertial>
     </link>
@@ -421,12 +421,12 @@
             <origin xyz="0 0 0" rpy="-1.57080 0 0"/>
             <geometry>
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