Commit message: update urdf

File: src/bopt_description/urdf/robot.urdf.xacro (robot description, xacro)
@@ -22,6 +22,6 @@
         </collision>
         <inertial>
-            <origin xyz="0 0 0" rpy="0 0 0"/>
-            <mass value="20.0"/>
+            <origin xyz="0 0 -0.2500" rpy="0 0 0"/>
+            <mass value="50.0"/>
             <inertia ixx="0.01" ixy="0.0" ixz="0.0"
                      iyy="0.01" iyz="0.0"
@@ -32,5 +32,5 @@
         <parent link="base_footprint"/>
         <child link="base_link"/>
-        <origin xyz="-1.2 0 0.350" rpy="0 0 0"/>
+        <origin xyz="0 0 0.300" rpy="0 0 0"/>
     </joint>
     <!-- ================================================================
@@ -66,6 +66,6 @@
         <origin xyz="0 0 0" rpy="0 0 0"/>
         <axis xyz="0 0 1"/>
-        <limit lower="-1.5708" upper="1.5708" effort="1" velocity="1"/>
-        <dynamics damping="0.1" friction="0.1"/>
+        <limit lower="-1.5708" upper="1.5708" effort="1000" velocity="2"/>
+        <dynamics damping="5" friction="1"/>
     </joint>
     <!-- Drive wheel -->
@@ -87,8 +87,8 @@
             <!-- mass=1 kg, solid cylinder r=0.05215 m, l=0.03 m -->
             <origin xyz="0 0 0" rpy="0 0 0"/>
-            <mass value="1.0"/>
-            <inertia ixx="0.01" ixy="0.0" ixz="0.0"
-                     iyy="0.01" iyz="0.0"
-                     izz="0.01"/>
+            <mass value="2.0"/>
+            <inertia ixx="0.02" ixy="0.0" ixz="0.0"
+                     iyy="0.02" iyz="0.0"
+                     izz="0.02"/>
         </inertial>
     </link>
@@ -98,5 +98,6 @@
         <origin xyz="0 0 -0.222" rpy="0 0 0"/>
         <axis xyz="0 1 0"/>
-        <dynamics damping="0.1" friction="0.1"/>
+        <limit lower="-3.1415" upper="3.1415" effort="1000" velocity="0.2"/>
+        <dynamics damping="5" friction="2"/>
     </joint>
     <!-- ================================================================
@@ -122,7 +123,7 @@
             <origin xyz="0 0 0" rpy="0 0 0"/>
             <mass value="1.0"/>
-            <inertia ixx="0.01" ixy="0.0" ixz="0.0"
-                     iyy="0.01" iyz="0.0"
-                     izz="0.01"/>
+            <inertia ixx="0.02" ixy="0.0" ixz="0.0"
+                     iyy="0.02" iyz="0.0"
+                     izz="0.02"/>
         </inertial>
     </link>
@@ -132,5 +133,5 @@
         <origin xyz="0 -0.255 -0.20515" rpy="0 0 0"/>
         <axis xyz="0 0 1"/>
-        <dynamics damping="0.1" friction="0.1"/>
+        <dynamics damping="5" friction="1"/>
     </joint>
     <!-- Caster assembly - left -->
@@ -153,7 +154,7 @@
             <origin xyz="0 0 0" rpy="0 0 0"/>
             <mass value="1.0"/>
-            <inertia ixx="0.01" ixy="0.0" ixz="0.0"
-                     iyy="0.01" iyz="0.0"
-                     izz="0.01"/>
+            <inertia ixx="0.02" ixy="0.0" ixz="0.0"
+                     iyy="0.02" iyz="0.0"
+                     izz="0.02"/>
         </inertial>
     </link>
@@ -163,5 +164,5 @@
         <origin xyz="0 0.255 -0.20515" rpy="0 0 0"/>
         <axis xyz="0 0 1"/>
-        <dynamics damping="0.1" friction="0.1"/>
+        <dynamics damping="5" friction="1"/>
     </joint>
     <!-- Caster wheel - right -->
@@ -184,7 +185,7 @@
             <origin xyz="0 0 0" rpy="0 0 0"/>
             <mass value="0.5"/>
-            <inertia ixx="0.01" ixy="0.0" ixz="0.0"
-                     iyy="0.01" iyz="0.0"
-                     izz="0.01"/>
+            <inertia ixx="0.02" ixy="0.0" ixz="0.0"
+                     iyy="0.02" iyz="0.0"
+                     izz="0.02"/>
         </inertial>
     </link>
@@ -194,5 +195,5 @@
         <origin xyz="0 0 -0.08105" rpy="0 0 0"/>
         <axis xyz="0 1 0"/>
-        <dynamics damping="0.1" friction="0.1"/>
+        <dynamics damping="5" friction="1"/>
     </joint>
     <!-- Caster wheel - left -->
@@ -215,7 +216,7 @@
             <origin xyz="0 0 0" rpy="0 0 0"/>
             <mass value="0.5"/>
-            <inertia ixx="0.01" ixy="0.0" ixz="0.0"
-                     iyy="0.01" iyz="0.0"
-                     izz="0.01"/>
+            <inertia ixx="0.02" ixy="0.0" ixz="0.0"
+                     iyy="0.02" iyz="0.0"
+                     izz="0.02"/>
         </inertial>
     </link>
@@ -225,5 +226,5 @@
         <origin xyz="0 0 -0.08105" rpy="0 0 0"/>
         <axis xyz="0 1 0"/>
-        <dynamics damping="0.1" friction="0.1"/>
+        <dynamics damping="5" friction="1"/>
     </joint>
     <!-- ================================================================
@@ -392,7 +393,7 @@
         </visual>
         <collision>
-            <origin xyz="0.22 0 0.1" rpy="0 0 0"/>
-            <geometry>
-                <box size="0.5 0.6 0.1"/>
+            <origin xyz="0 0 0" rpy="0 0 0"/>
+            <geometry>
+                <mesh filename="file:///home/jkw/bopt_ws/install/bopt_description/share/bopt_description/meshes/visual/front.stl"/>
             </geometry>
         </collision>
@@ -400,8 +401,8 @@
             <!-- mass=3 kg, box 0.1 x 0.1 x 0.1 m -->
             <origin xyz="0 0 0" rpy="0 0 0"/>
-            <mass value="3.0"/>
-            <inertia ixx="0.01" ixy="0.0" ixz="0.0"
-                     iyy="0.01" iyz="0.0"
-                     izz="0.01"/>
+            <mass value="15"/>
+            <inertia ixx="0.02" ixy="0.0" ixz="0.0"
+                     iyy="0.02" iyz="0.0"
+                     izz="0.02"/>
         </inertial>
     </link>
@@ -411,5 +412,6 @@
         <origin xyz="0.477 0 -0.265" rpy="0 0 0"/>
         <axis xyz="0 0 1"/>
-        <limit lower="0" upper="0.095" effort="1000000" velocity="2.0"/>
+        <limit lower="0" upper="0.095" effort="30000" velocity="0.03"/>
+        <dynamics damping="200" friction="20"/>
     </joint>
     <!-- ================================================================
@@ -434,5 +436,5 @@
             <!-- mass=3 kg, solid cylinder r=0.175 m, l=0.1 m -->
             <origin xyz="0.148 0 0" rpy="0 0 0"/>
-            <mass value="1"/>
+            <mass value="0.1"/>
             <inertia ixx="0.01" ixy="0.0" ixz="0.0"
                      iyy="0.01" iyz="0.0"
@@ -446,5 +448,5 @@
         <axis xyz="0 1 0"/>
         <limit lower="0" upper="0.7854" effort="50" velocity="2"/>
-        <dynamics damping="0.1" friction="0.1"/>
+        <dynamics damping="5" friction="1"/>
     </joint>
     <link name="front_wheel_shaft_right">
@@ -465,5 +467,5 @@
             <!-- mass=3 kg, solid cylinder r=0.175 m, l=0.1 m -->
             <origin xyz="0.148 0 0" rpy="0 0 0"/>
-            <mass value="1"/>
+            <mass value="0.1"/>
             <inertia ixx="0.01" ixy="0.0" ixz="0.0"
                      iyy="0.01" iyz="0.0"
@@ -477,5 +479,5 @@
         <axis xyz="0 1 0"/>
         <limit lower="0" upper="0.7854" effort="50" velocity="2"/>
-        <dynamics damping="0.1" friction="0.1"/>
+        <dynamics damping="5" friction="1"/>
     </joint>
     <!-- Front wheel - right -->
@@ -497,5 +499,5 @@
             <!-- mass=3 kg, solid cylinder r=0.175 m, l=0.1 m -->
             <origin xyz="0 0 0" rpy="0 0 0"/>
-            <mass value="3.0"/>
+            <mass value="1.0"/>
             <inertia ixx="0.01" ixy="0.0" ixz="0.0"
                      iyy="0.01" iyz="0.0"
@@ -508,5 +510,5 @@
         <origin xyz="0.1488 -0.067 -0.0013" rpy="0 0 0"/>
         <axis xyz="0 1 0"/>
-        <dynamics damping="0.1" friction="0.1"/>
+        <dynamics damping="5" friction="1"/>
     </joint>
     <!-- Front wheel - left -->
@@ -528,5 +530,5 @@
             <!-- mass=3 kg, solid cylinder r=0.175 m, l=0.1 m -->
             <origin xyz="0 0 0" rpy="0 0 0"/>
-            <mass value="3.0"/>
+            <mass value="1.0"/>
             <inertia ixx="0.01" ixy="0.0" ixz="0.0"
                      iyy="0.01" iyz="0.0"
@@ -539,5 +541,5 @@
         <origin xyz="0.1488 0.077 -0.0013" rpy="0 0 0"/>
         <axis xyz="0 1 0"/>
-        <dynamics damping="0.1" friction="0.1"/>
+        <dynamics damping="5" friction="1"/>
     </joint>
     <gazebo reference="base_link">
@@ -592,3 +594,48 @@
         <material>Gazebo/Black</material>
     </gazebo>
+    <gazebo reference="drive_wheel">
+        <mu1>1.5</mu1>
+        <mu2>1.5</mu2>
+    </gazebo>
+    <gazebo reference="caster_wheel_left">
+        <mu1>1.2</mu1>
+        <mu2>1.2</mu2>
+    </gazebo>
+    <gazebo reference="caster_wheel_right">
+        <mu1>1.2</mu1>
+        <mu2>1.2</mu2>
+    </gazebo>
+    <gazebo reference="front_wheel_left">
+        <mu1>1.2</mu1>
+        <mu2>1.2</mu2>
+    </gazebo>
+    <gazebo reference="front_wheel_right">
+        <mu1>1.2</mu1>
+        <mu2>1.2</mu2>
+    </gazebo>
+    <ros2_control name="GazeboSystem" type="system">
+        <hardware>
+            <plugin>gazebo_ros2_control/GazeboSystem</plugin>
+        </hardware>
+        <joint name="drive_wheel_Ass_joint">
+            <command_interface name="position"/>
+            <state_interface name="position"/>
+            <state_interface name="velocity"/>
+        </joint>
+        <joint name="drive_wheel_joint">
+            <command_interface name="velocity"/>
+            <state_interface name="position"/>
+            <state_interface name="velocity"/>
+        </joint>
+        <joint name="front_lift_joint">
+            <command_interface name="position"/>
+            <state_interface name="position"/>
+            <state_interface name="velocity"/>
+        </joint>
+    </ros2_control>
+    <gazebo>
+        <plugin filename="libgazebo_ros2_control.so" name="gazebo_ros2_control">
+            <parameters>$(find bopt_description)/config/controllers.yaml</parameters>
+        </plugin>
+    </gazebo>
 </robot>

Commit message: update

File: src/bopt_description/urdf/robot.urdf.xacro (robot description, xacro)
@@ -1,3 +1,8 @@
 <?xml version="1.0"?>
+<!--
+  BOPT Robot URDF Description
+  This file defines the physical properties, joints, links, and sensor locations of the bopt_robot.
+  It also includes Gazebo simulation materials and ros2_control interfaces.
+-->
 <robot xmlns:xacro="http://www.ros.org/wiki/xacro" name="bopt_robot">
     <xacro:include filename="materials.xacro"/>
@@ -47,5 +52,5 @@
         </visual>
         <collision>
-            <origin xyz="0 0 00" rpy="0 0 0"/>
+            <origin xyz="0 0 0" rpy="0 0 0"/>
             <geometry>
                 <mesh filename="file:///home/jkw/bopt_ws/install/bopt_description/share/bopt_description/meshes/visual/drive_wheel_ass.stl"/>
@@ -85,5 +90,5 @@
         </collision>
         <inertial>
-            <!-- mass=1 kg, solid cylinder r=0.05215 m, l=0.03 m -->
+            <!-- mass=2.0 kg, solid cylinder r=0.05215 m, l=0.03 m -->
             <origin xyz="0 0 0" rpy="0 0 0"/>
             <mass value="2.0"/>
@@ -193,5 +198,5 @@
         <parent link="caster_wheel_ass_right"/>
         <child link="caster_wheel_right"/>
-        <origin xyz="0 0 -0.08105" rpy="0 0 0"/>
+        <origin xyz="0 0 -0.08109" rpy="0 0 0"/>
         <axis xyz="0 1 0"/>
         <dynamics damping="5" friction="1"/>
@@ -224,5 +229,5 @@
         <parent link="caster_wheel_ass_left"/>
         <child link="caster_wheel_left"/>
-        <origin xyz="0 0 -0.08105" rpy="0 0 0"/>
+        <origin xyz="0 0 -0.08109" rpy="0 0 0"/>
         <axis xyz="0 1 0"/>
         <dynamics damping="5" friction="1"/>
@@ -399,6 +404,6 @@
         </collision>
         <inertial>
-            <!-- mass=3 kg, box 0.1 x 0.1 x 0.1 m -->
-            <origin xyz="0 0 0" rpy="0 0 0"/>
+            <!-- mass=15 kg, box 0.1 x 0.1 x 0.1 m -->
+            <origin xyz="0.477 0 0" rpy="0 0 0"/>
             <mass value="15"/>
             <inertia ixx="0.02" ixy="0.0" ixz="0.0"
@@ -410,7 +415,7 @@
         <parent link="base_link"/>
         <child link="front_lift_link"/>
-        <origin xyz="0.477 0 -0.265" rpy="0 0 0"/>
+        <origin xyz="0.377 0 -0.265" rpy="0 0 0"/>
         <axis xyz="0 0 1"/>
-        <limit lower="0" upper="0.095" effort="30000" velocity="0.03"/>
+        <limit lower="0" upper="0.095" effort="30000" velocity="0.003"/>
         <dynamics damping="200" friction="20"/>
     </joint>
@@ -418,12 +423,74 @@
          FRONT WHEELS
          ================================================================ -->
-    <!--front wheel shaft- left -->
+    <!-- Front socket - left (Prismatic movement) -->
+    <link name="front_socket_left">
+        <visual>
+            <origin xyz="0 0 0" rpy="0 0 0"/>
+            <geometry>
+                <mesh filename="file:///home/jkw/bopt_ws/install/bopt_description/share/bopt_description/meshes/visual/front_socket.stl"/>
+            </geometry>
+            <material name="gray"/>
+        </visual>
+        <collision>
+            <origin xyz="0 0 0" rpy="0 0 0"/>
+            <geometry>
+                <mesh filename="file:///home/jkw/bopt_ws/install/bopt_description/share/bopt_description/meshes/visual/front_socket.stl"/>
+            </geometry>
+        </collision>
+        <inertial>
+            <origin xyz="0 0 0" rpy="0 0 0"/>
+            <mass value="0.1"/>
+            <inertia ixx="0.001" ixy="0.0" ixz="0.0"
+                     iyy="0.001" iyz="0.0"
+                     izz="0.001"/>
+        </inertial>
+    </link>
+    <joint name="front_socket_left_joint" type="prismatic">
+        <parent link="front_lift_link"/>
+        <child link="front_socket_left"/>
+        <origin xyz="0.876075 0.2565 0.0176" rpy="0 0 0"/>
+        <axis xyz="1 0 0"/>
+        <limit lower="0" upper="0.01068" effort="50" velocity="2"/>
+        <dynamics damping="1.5" friction="2"/>
+    </joint>
+    <!-- Front socket - right (Prismatic movement) -->
+    <link name="front_socket_right">
+        <visual>
+            <origin xyz="0 0 0" rpy="0 0 0"/>
+            <geometry>
+                <mesh filename="file:///home/jkw/bopt_ws/install/bopt_description/share/bopt_description/meshes/visual/front_socket.stl"/>
+            </geometry>
+            <material name="gray"/>
+        </visual>
+        <collision>
+            <origin xyz="0 0 0" rpy="0 0 0"/>
+            <geometry>
+                <mesh filename="file:///home/jkw/bopt_ws/install/bopt_description/share/bopt_description/meshes/visual/front_socket.stl"/>
+            </geometry>
+        </collision>
+        <inertial>
+            <origin xyz="0 0 0" rpy="0 0 0"/>
+            <mass value="0.1"/>
+            <inertia ixx="0.001" ixy="0.0" ixz="0.0"
+                     iyy="0.001" iyz="0.0"
+                     izz="0.001"/>
+        </inertial>
+    </link>
+    <joint name="front_socket_right_joint" type="prismatic">
+        <parent link="front_lift_link"/>
+        <child link="front_socket_right"/>
+        <origin xyz="0.87605 -0.1085 0.0176" rpy="0 0 0"/>
+        <axis xyz="1 0 0"/>
+        <limit lower="0" upper="0.01068" effort="50" velocity="2"/>
+        <dynamics damping="1.5" friction="2"/>
+    </joint>
+    <!-- Front wheel shaft - left -->
     <link name="front_wheel_shaft_left">
         <visual>
-            <origin xyz="0 0 0" rpy="-1.57080 0 0"/>
+            <origin xyz="0 0 0" rpy="1.5708 0 0"/>
             <geometry>
                 <mesh filename="file:///home/jkw/bopt_ws/install/bopt_description/share/bopt_description/meshes/visual/front_wheel_shaft.stl"/>
             </geometry>
-            <material name="black"/>
+            <material name="gray"/>
         </visual>
         <collision>
@@ -434,7 +501,6 @@
         </collision>
         <inertial>
-            <!-- mass=3 kg, solid cylinder r=0.175 m, l=0.1 m -->
             <origin xyz="0.148 0 0" rpy="0 0 0"/>
-            <mass value="0.1"/>
+            <mass value="1"/>
             <inertia ixx="0.01" ixy="0.0" ixz="0.0"
                      iyy="0.01" iyz="0.0"
@@ -443,11 +509,12 @@
     </link>
     <joint name="front_wheel_shaft_left_joint" type="revolute">
-        <parent link="front_lift_link"/>
+        <parent link="front_socket_left"/>
         <child link="front_wheel_shaft_left"/>
-        <origin xyz="0.9211 0.1055 -0.01758" rpy="0 0 0"/>
+        <origin xyz="0.045125 -0.008 0" rpy="0 0.259 0"/>
         <axis xyz="0 1 0"/>
-        <limit lower="0" upper="0.7854" effort="50" velocity="2"/>
-        <dynamics damping="5" friction="1"/>
-    </joint>
+        <limit lower="0" upper="0.785" effort="50" velocity="2"/>
+        <dynamics damping="3" friction="2"/>
+    </joint>
+    <!-- Front wheel shaft - right -->
     <link name="front_wheel_shaft_right">
         <visual>
@@ -456,5 +523,5 @@
                 <mesh filename="file:///home/jkw/bopt_ws/install/bopt_description/share/bopt_description/meshes/visual/front_wheel_shaft.stl"/>
             </geometry>
-            <material name="black"/>
+            <material name="gray"/>
         </visual>
         <collision>
@@ -465,7 +532,6 @@
         </collision>
         <inertial>
-            <!-- mass=3 kg, solid cylinder r=0.175 m, l=0.1 m -->
             <origin xyz="0.148 0 0" rpy="0 0 0"/>
-            <mass value="0.1"/>
+            <mass value="1"/>
             <inertia ixx="0.01" ixy="0.0" ixz="0.0"
                      iyy="0.01" iyz="0.0"
@@ -474,10 +540,10 @@
     </link>
     <joint name="front_wheel_shaft_right_joint" type="revolute">
-        <parent link="front_lift_link"/>
+        <parent link="front_socket_right"/>
         <child link="front_wheel_shaft_right"/>
-        <origin xyz="0.9211 -0.1135 -0.01758" rpy="0 0 0"/>
+        <origin xyz="0.045125 -0.008 0" rpy="0 0.259 0"/>
         <axis xyz="0 1 0"/>
-        <limit lower="0" upper="0.7854" effort="50" velocity="2"/>
-        <dynamics damping="5" friction="1"/>
+        <limit lower="0" upper="0.785" effort="50" velocity="2"/>
+        <dynamics damping="3" friction="2"/>
     </joint>
     <!-- Front wheel - right -->
@@ -497,7 +563,7 @@
         </collision>
         <inertial>
-            <!-- mass=3 kg, solid cylinder r=0.175 m, l=0.1 m -->
-            <origin xyz="0 0 0" rpy="0 0 0"/>
-            <mass value="1.0"/>
+            <!-- mass=2 kg, solid cylinder r=0.0425 m, l=0.110 m -->
+            <origin xyz="0 0 0" rpy="0 0 0"/>
+            <mass value="2.0"/>
             <inertia ixx="0.01" ixy="0.0" ixz="0.0"
                      iyy="0.01" iyz="0.0"
@@ -508,5 +574,5 @@
         <parent link="front_wheel_shaft_right"/>
         <child link="front_wheel_right"/>
-        <origin xyz="0.1488 -0.067 -0.0013" rpy="0 0 0"/>
+        <origin xyz="0.1488 -0.067 -0.0025435" rpy="0 0 0"/>
         <axis xyz="0 1 0"/>
         <dynamics damping="5" friction="1"/>
@@ -528,7 +594,7 @@
         </collision>
         <inertial>
-            <!-- mass=3 kg, solid cylinder r=0.175 m, l=0.1 m -->
-            <origin xyz="0 0 0" rpy="0 0 0"/>
-            <mass value="1.0"/>
+            <!-- mass=2 kg, solid cylinder r=0.0425 m, l=0.110 m -->
+            <origin xyz="0 0 0" rpy="0 0 0"/>
+            <mass value="2.0"/>
             <inertia ixx="0.01" ixy="0.0" ixz="0.0"
                      iyy="0.01" iyz="0.0"
@@ -539,8 +605,11 @@
         <parent link="front_wheel_shaft_left"/>
         <child link="front_wheel_left"/>
-        <origin xyz="0.1488 0.077 -0.0013" rpy="0 0 0"/>
+        <origin xyz="0.1488 -0.067 -0.0025435" rpy="0 0 0"/>
         <axis xyz="0 1 0"/>
         <dynamics damping="5" friction="1"/>
     </joint>
+    <!-- ================================================================
+         GAZEBO MATERIALS
+         ================================================================ -->
     <gazebo reference="base_link">
         <material>Gazebo/Blue</material>
@@ -593,4 +662,15 @@
     <gazebo reference="front_wheel_left">
         <material>Gazebo/Black</material>
+    </gazebo>
+    <!-- ================================================================
+         GAZEBO FRICTION PROPERTIES
+         ================================================================ -->
+    <gazebo reference="front_socket_left_joint">
+        <spring_reference>0.025</spring_reference>
+        <spring_stiffness>5000</spring_stiffness>
+    </gazebo>
+     <gazebo reference="front_socket_right_joint">
+        <spring_reference>0.025</spring_reference>
+        <spring_stiffness>5000</spring_stiffness>
     </gazebo>
     <gazebo reference="drive_wheel">
@@ -614,4 +694,17 @@
         <mu2>1.2</mu2>
     </gazebo>
+    <gazebo reference="front_socket_left_joint">
+        <implicit_spring_damper>true</implicit_spring_damper>
+        <spring_reference>0.025</spring_reference>
+        <spring_stiffness>3000</spring_stiffness>
+    </gazebo>
+    <gazebo reference="front_socket_right_joint">
+        <implicit_spring_damper>true</implicit_spring_damper>
+        <spring_reference>0.025</spring_reference>
+        <spring_stiffness>3000</spring_stiffness>
+    </gazebo>
+    <!-- ================================================================
+         ROS2 CONTROL PLUGINS AND INTERFACES
+         ================================================================ -->
     <ros2_control name="GazeboSystem" type="system">
         <hardware>
@@ -619,15 +712,24 @@
         </hardware>
         <joint name="drive_wheel_Ass_joint">
-            <command_interface name="position"/>
+            <command_interface name="position">
+                <param name="min">-1.512</param>
+                <param name="max">1.512</param>
+            </command_interface>
             <state_interface name="position"/>
             <state_interface name="velocity"/>
         </joint>
         <joint name="drive_wheel_joint">
-            <command_interface name="velocity"/>
+            <command_interface name="velocity">
+                <param name="min">-3.0</param>
+                <param name="max">3.0</param>
+            </command_interface>
             <state_interface name="position"/>
             <state_interface name="velocity"/>
         </joint>
         <joint name="front_lift_joint">
-            <command_interface name="position"/>
+            <command_interface name="position">
+                <param name="min">0.0</param>
+                <param name="max">0.095</param>
+            </command_interface>
             <state_interface name="position"/>
             <state_interface name="velocity"/>
