Commit message: i dont know

File: src/bopt_description/urdf/robot.urdf.xacro (robot description, xacro)
@@ -103,5 +103,4 @@
         <origin xyz="0 0 -0.222" rpy="0 0 0"/>
         <axis xyz="0 1 0"/>
-        <limit lower="-3.1415" upper="3.1415" effort="1000" velocity="0.2"/>
         <dynamics damping="5" friction="2"/>
     </joint>
@@ -405,5 +404,5 @@
         <inertial>
             <!-- mass=15 kg, box 0.1 x 0.1 x 0.1 m -->
-            <origin xyz="0.477 0 0" rpy="0 0 0"/>
+            <origin xyz="0 0 0" rpy="0 0 0"/>
             <mass value="15"/>
             <inertia ixx="0.02" ixy="0.0" ixz="0.0"
@@ -415,8 +414,8 @@
         <parent link="base_link"/>
         <child link="front_lift_link"/>
-        <origin xyz="0.377 0 -0.265" rpy="0 0 0"/>
+        <origin xyz="0.477 0 -0.265" rpy="0 0 0"/>
         <axis xyz="0 0 1"/>
-        <limit lower="0" upper="0.095" effort="30000" velocity="0.003"/>
-        <dynamics damping="200" friction="20"/>
+        <limit lower="0" upper="0.095" effort="30000" velocity="0.03"/>
+        <dynamics damping="50" friction="10"/>
     </joint>
     <!-- ================================================================
@@ -451,6 +450,6 @@
         <origin xyz="0.876075 0.2565 0.0176" rpy="0 0 0"/>
         <axis xyz="1 0 0"/>
-        <limit lower="0" upper="0.01068" effort="50" velocity="2"/>
-        <dynamics damping="1.5" friction="2"/>
+        <limit lower="0" upper="0.00868" effort="50" velocity="2"/>
+        <dynamics damping="5.0" friction="2"/>
     </joint>
     <!-- Front socket - right (Prismatic movement) -->
@@ -482,6 +481,6 @@
         <origin xyz="0.87605 -0.1085 0.0176" rpy="0 0 0"/>
         <axis xyz="1 0 0"/>
-        <limit lower="0" upper="0.01068" effort="50" velocity="2"/>
-        <dynamics damping="1.5" friction="2"/>
+        <limit lower="0" upper="0.00868" effort="50" velocity="2"/>
+        <dynamics damping="5.0" friction="2"/>
     </joint>
     <!-- Front wheel shaft - left -->
@@ -495,7 +494,7 @@
         </visual>
         <collision>
-            <origin xyz="0 0 0" rpy="0 0 0"/>
-            <geometry>
-                <box size="0.14 0.05 0.05"/>
+            <origin xyz="0 0 0" rpy="1.5708 0 0"/>
+            <geometry>
+                <mesh filename="file:///home/jkw/bopt_ws/install/bopt_description/share/bopt_description/meshes/visual/front_wheel_shaft.stl"/>
             </geometry>
         </collision>
@@ -514,5 +513,5 @@
         <axis xyz="0 1 0"/>
         <limit lower="0" upper="0.785" effort="50" velocity="2"/>
-        <dynamics damping="3" friction="2"/>
+        <dynamics damping="5.0" friction="1"/>
     </joint>
     <!-- Front wheel shaft - right -->
@@ -526,7 +525,7 @@
         </visual>
         <collision>
-            <origin xyz="0 0 0" rpy="0 0 0"/>
-            <geometry>
-                <box size="0.14 0.05 0.05"/>
+            <origin xyz="0 0 0" rpy="1.5708 0 0"/>
+            <geometry>
+                <mesh filename="file:///home/jkw/bopt_ws/install/bopt_description/share/bopt_description/meshes/visual/front_wheel_shaft.stl"/>
             </geometry>
         </collision>
@@ -545,5 +544,5 @@
         <axis xyz="0 1 0"/>
         <limit lower="0" upper="0.785" effort="50" velocity="2"/>
-        <dynamics damping="3" friction="2"/>
+        <dynamics damping="5.0" friction="1"/>
     </joint>
     <!-- Front wheel - right -->
@@ -574,5 +573,5 @@
         <parent link="front_wheel_shaft_right"/>
         <child link="front_wheel_right"/>
-        <origin xyz="0.1488 -0.067 -0.0025435" rpy="0 0 0"/>
+        <origin xyz="0.1488 -0.067 -0.0025435" rpy="0 -0.259 0"/>
         <axis xyz="0 1 0"/>
         <dynamics damping="5" friction="1"/>
@@ -605,5 +604,5 @@
         <parent link="front_wheel_shaft_left"/>
         <child link="front_wheel_left"/>
-        <origin xyz="0.1488 -0.067 -0.0025435" rpy="0 0 0"/>
+        <origin xyz="0.1488 -0.067 -0.0025435" rpy="0 -0.259 0"/>
         <axis xyz="0 1 0"/>
         <dynamics damping="5" friction="1"/>
@@ -666,12 +665,4 @@
          GAZEBO FRICTION PROPERTIES
          ================================================================ -->
-    <gazebo reference="front_socket_left_joint">
-        <spring_reference>0.025</spring_reference>
-        <spring_stiffness>5000</spring_stiffness>
-    </gazebo>
-     <gazebo reference="front_socket_right_joint">
-        <spring_reference>0.025</spring_reference>
-        <spring_stiffness>5000</spring_stiffness>
-    </gazebo>
     <gazebo reference="drive_wheel">
         <mu1>1.5</mu1>
@@ -693,14 +684,4 @@
         <mu1>1.2</mu1>
         <mu2>1.2</mu2>
-    </gazebo>
-    <gazebo reference="front_socket_left_joint">
-        <implicit_spring_damper>true</implicit_spring_damper>
-        <spring_reference>0.025</spring_reference>
-        <spring_stiffness>3000</spring_stiffness>
-    </gazebo>
-    <gazebo reference="front_socket_right_joint">
-        <implicit_spring_damper>true</implicit_spring_damper>
-        <spring_reference>0.025</spring_reference>
-        <spring_stiffness>3000</spring_stiffness>
     </gazebo>
     <!-- ================================================================

Commit message: update urdf and controller

File: src/bopt_description/urdf/robot.urdf.xacro (robot description, xacro)
@@ -71,6 +71,6 @@
         <origin xyz="0 0 0" rpy="0 0 0"/>
         <axis xyz="0 0 1"/>
-        <limit lower="-1.5708" upper="1.5708" effort="1000" velocity="2"/>
-        <dynamics damping="5" friction="1"/>
+        <limit lower="-3.14159" upper="3.14159" effort="1000" velocity="2"/>
+        <dynamics damping="5" friction="0.1"/>
     </joint>
     <!-- Drive wheel -->
@@ -84,11 +84,10 @@
         </visual>
         <collision>
-            <origin xyz="0 0 0" rpy="0 0 0"/>
-            <geometry>
-                <mesh filename="file:///home/jkw/bopt_ws/install/bopt_description/share/bopt_description/meshes/visual/drive_wheel.stl"/>
-            </geometry>
-        </collision>
-        <inertial>
-            <!-- mass=2.0 kg, solid cylinder r=0.05215 m, l=0.03 m -->
+            <origin xyz="0 0 0" rpy="1.5708 0 0"/>
+            <geometry>
+                <cylinder radius="0.115" length="0.074"/>
+            </geometry>
+        </collision>
+        <inertial>
             <origin xyz="0 0 0" rpy="0 0 0"/>
             <mass value="2.0"/>
@@ -101,7 +100,7 @@
         <parent link="drive_wheel_Ass"/>
         <child link="drive_wheel"/>
-        <origin xyz="0 0 -0.222" rpy="0 0 0"/>
+        <origin xyz="0 0 -0.223" rpy="0 0 0"/>
         <axis xyz="0 1 0"/>
-        <dynamics damping="5" friction="2"/>
+        <dynamics damping="5" friction="0.2"/>
     </joint>
     <!-- ================================================================
@@ -137,5 +136,5 @@
         <origin xyz="0 -0.255 -0.20515" rpy="0 0 0"/>
         <axis xyz="0 0 1"/>
-        <dynamics damping="5" friction="1"/>
+        <dynamics damping="5" friction="0.1"/>
     </joint>
     <!-- Caster assembly - left -->
@@ -168,5 +167,5 @@
         <origin xyz="0 0.255 -0.20515" rpy="0 0 0"/>
         <axis xyz="0 0 1"/>
-        <dynamics damping="5" friction="1"/>
+        <dynamics damping="5" friction="0.1"/>
     </joint>
     <!-- Caster wheel - right -->
@@ -180,11 +179,10 @@
         </visual>
         <collision>
-            <origin xyz="0 0 0" rpy="0 0 0"/>
-            <geometry>
-                <mesh filename="file:///home/jkw/bopt_ws/install/bopt_description/share/bopt_description/meshes/visual/casster_wheel.stl"/>
-            </geometry>
-        </collision>
-        <inertial>
-            <!-- mass=0.5 kg, solid cylinder r=0.05215 m, l=0.03 m -->
+            <origin xyz="0 0 0" rpy="1.5708 0 0"/>
+            <geometry>
+                <cylinder radius="0.050" length="0.060"/>
+            </geometry>
+        </collision>
+        <inertial>
             <origin xyz="0 0 0" rpy="0 0 0"/>
             <mass value="0.5"/>
@@ -197,7 +195,7 @@
         <parent link="caster_wheel_ass_right"/>
         <child link="caster_wheel_right"/>
-        <origin xyz="0 0 -0.08109" rpy="0 0 0"/>
+        <origin xyz="0 0 -0.0827" rpy="0 0 0"/>
         <axis xyz="0 1 0"/>
-        <dynamics damping="5" friction="1"/>
+        <dynamics damping="5" friction="0.1"/>
     </joint>
     <!-- Caster wheel - left -->
@@ -211,11 +209,10 @@
         </visual>
         <collision>
-            <origin xyz="0 0 0" rpy="0 0 0"/>
-            <geometry>
-                <mesh filename="file:///home/jkw/bopt_ws/install/bopt_description/share/bopt_description/meshes/visual/casster_wheel.stl"/>
-            </geometry>
-        </collision>
-        <inertial>
-            <!-- mass=0.5 kg, solid cylinder r=0.05215 m, l=0.03 m -->
+            <origin xyz="0 0 0" rpy="1.5708 0 0"/>
+            <geometry>
+                <cylinder radius="0.050" length="0.060"/>
+            </geometry>
+        </collision>
+        <inertial>
             <origin xyz="0 0 0" rpy="0 0 0"/>
             <mass value="0.5"/>
@@ -228,7 +225,7 @@
         <parent link="caster_wheel_ass_left"/>
         <child link="caster_wheel_left"/>
-        <origin xyz="0 0 -0.08109" rpy="0 0 0"/>
+        <origin xyz="0 0 -0.0827" rpy="0 0 0"/>
         <axis xyz="0 1 0"/>
-        <dynamics damping="5" friction="1"/>
+        <dynamics damping="5" friction="0.1"/>
     </joint>
     <!-- ================================================================
@@ -404,5 +401,5 @@
         <inertial>
             <!-- mass=15 kg, box 0.1 x 0.1 x 0.1 m -->
-            <origin xyz="0 0 0" rpy="0 0 0"/>
+            <origin xyz="0.477 0 0" rpy="0 0 0"/>
             <mass value="15"/>
             <inertia ixx="0.02" ixy="0.0" ixz="0.0"
@@ -513,5 +510,5 @@
         <axis xyz="0 1 0"/>
         <limit lower="0" upper="0.785" effort="50" velocity="2"/>
-        <dynamics damping="5.0" friction="1"/>
+        <dynamics damping="5.0" friction="0.1"/>
     </joint>
     <!-- Front wheel shaft - right -->
@@ -544,5 +541,5 @@
         <axis xyz="0 1 0"/>
         <limit lower="0" upper="0.785" effort="50" velocity="2"/>
-        <dynamics damping="5.0" friction="1"/>
+        <dynamics damping="5.0" friction="0.1"/>
     </joint>
     <!-- Front wheel - right -->
@@ -556,7 +553,7 @@
         </visual>
         <collision>
-            <origin xyz="0 0 0" rpy="0 0 0"/>
-            <geometry>
-                <mesh filename="file:///home/jkw/bopt_ws/install/bopt_description/share/bopt_description/meshes/visual/front_wheel.stl"/>
+            <origin xyz="0 0 0" rpy="1.5708 0 0"/>
+            <geometry>
+                <cylinder radius="0.0425" length="0.110"/>
             </geometry>
         </collision>
@@ -575,5 +572,5 @@
         <origin xyz="0.1488 -0.067 -0.0025435" rpy="0 -0.259 0"/>
         <axis xyz="0 1 0"/>
-        <dynamics damping="5" friction="1"/>
+        <dynamics damping="5" friction="0.1"/>
     </joint>
     <!-- Front wheel - left -->
@@ -587,7 +584,7 @@
         </visual>
         <collision>
-            <origin xyz="0 0 0" rpy="0 0 0"/>
-            <geometry>
-                <mesh filename="file:///home/jkw/bopt_ws/install/bopt_description/share/bopt_description/meshes/visual/front_wheel.stl"/>
+            <origin xyz="0 0 0" rpy="1.5708 0 0"/>
+            <geometry>
+                <cylinder radius="0.0425" length="0.110"/>
             </geometry>
         </collision>
@@ -606,5 +603,5 @@
         <origin xyz="0.1488 -0.067 -0.0025435" rpy="0 -0.259 0"/>
         <axis xyz="0 1 0"/>
-        <dynamics damping="5" friction="1"/>
+        <dynamics damping="5" friction="0.1"/>
     </joint>
     <!-- ================================================================
@@ -670,18 +667,18 @@
     </gazebo>
     <gazebo reference="caster_wheel_left">
-        <mu1>1.2</mu1>
-        <mu2>1.2</mu2>
+        <mu1>1.5</mu1>
+        <mu2>1.5</mu2>
     </gazebo>
     <gazebo reference="caster_wheel_right">
-        <mu1>1.2</mu1>
-        <mu2>1.2</mu2>
+        <mu1>1.5</mu1>
+        <mu2>1.5</mu2>
     </gazebo>
     <gazebo reference="front_wheel_left">
-        <mu1>1.2</mu1>
-        <mu2>1.2</mu2>
+        <mu1>1.0</mu1>
+        <mu2>1.0</mu2>
     </gazebo>
     <gazebo reference="front_wheel_right">
-        <mu1>1.2</mu1>
-        <mu2>1.2</mu2>
+        <mu1>1.0</mu1>
+        <mu2>1.0</mu2>
     </gazebo>
     <!-- ================================================================
@@ -694,6 +691,6 @@
         <joint name="drive_wheel_Ass_joint">
             <command_interface name="position">
-                <param name="min">-1.512</param>
-                <param name="max">1.512</param>
+                <param name="min">-3.14159</param>
+                <param name="max">3.14159</param>
             </command_interface>
             <state_interface name="position"/>
@@ -716,4 +713,20 @@
             <state_interface name="velocity"/>
         </joint>
+        <joint name="caster_wheel_ass_joint_left">
+            <state_interface name="position"/>
+            <state_interface name="velocity"/>
+        </joint>
+        <joint name="caster_wheel_ass_joint_right">
+            <state_interface name="position"/>
+            <state_interface name="velocity"/>
+        </joint>
+        <joint name="front_wheel_left_joint">
+            <state_interface name="position"/>
+            <state_interface name="velocity"/>
+        </joint>
+        <joint name="front_wheel_right_joint">
+            <state_interface name="position"/>
+            <state_interface name="velocity"/>
+        </joint>
     </ros2_control>
     <gazebo>

Commit message: urdf file

File: src/bopt_description/urdf/robot.urdf.xacro (robot description, xacro)
@@ -1,8 +1,3 @@
 <?xml version="1.0"?>
-<!--
-  BOPT Robot URDF Description
-  This file defines the physical properties, joints, links, and sensor locations of the bopt_robot.
-  It also includes Gazebo simulation materials and ros2_control interfaces.
--->
 <robot xmlns:xacro="http://www.ros.org/wiki/xacro" name="bopt_robot">
     <xacro:include filename="materials.xacro"/>
@@ -58,5 +53,4 @@
         </collision>
         <inertial>
-            <!-- mass=2 kg, box 0.3 x 0.3 x 0.1 m -->
             <origin xyz="0 0 0" rpy="0 0 0"/>
             <mass value="2.0"/>
@@ -123,5 +117,4 @@
         </collision>
         <inertial>
-            <!-- mass=1 kg, box 0.3 x 0.3 x 0.1 m -->
             <origin xyz="0 0 0" rpy="0 0 0"/>
             <mass value="1.0"/>
@@ -154,5 +147,4 @@
         </collision>
         <inertial>
-            <!-- mass=1 kg, box 0.3 x 0.3 x 0.1 m -->
             <origin xyz="0 0 0" rpy="0 0 0"/>
             <mass value="1.0"/>
@@ -248,5 +240,4 @@
         </collision>
         <inertial>
-            <!-- mass=0.2 kg, box 0.1 x 0.1 x 0.1 m -->
             <origin xyz="0 0 0" rpy="0 0 0"/>
             <mass value="0.2"/>
@@ -277,5 +268,4 @@
         </collision>
         <inertial>
-            <!-- mass=0.2 kg, box 0.1 x 0.1 x 0.1 m -->
             <origin xyz="0 0 0" rpy="0 0 0"/>
             <mass value="0.2"/>
@@ -309,5 +299,4 @@
         </collision>
         <inertial>
-            <!-- mass=0.2 kg, box 0.1 x 0.1 x 0.1 m -->
             <origin xyz="0 0 0" rpy="0 0 0"/>
             <mass value="0.2"/>
@@ -338,5 +327,4 @@
         </collision>
         <inertial>
-            <!-- mass=0.2 kg, box 0.1 x 0.1 x 0.1 m -->
             <origin xyz="0 0 0" rpy="0 0 0"/>
             <mass value="0.2"/>
@@ -369,5 +357,4 @@
         </collision>
         <inertial>
-            <!-- mass=0.5 kg, box 0.1 x 0.1 x 0.1 m -->
             <origin xyz="0 0 0" rpy="0 0 0"/>
             <mass value="0.5"/>
@@ -400,5 +387,4 @@
         </collision>
         <inertial>
-            <!-- mass=15 kg, box 0.1 x 0.1 x 0.1 m -->
             <origin xyz="0.477 0 0" rpy="0 0 0"/>
             <mass value="15"/>
@@ -559,5 +545,4 @@
         </collision>
         <inertial>
-            <!-- mass=2 kg, solid cylinder r=0.0425 m, l=0.110 m -->
             <origin xyz="0 0 0" rpy="0 0 0"/>
             <mass value="2.0"/>
@@ -586,9 +571,8 @@
             <origin xyz="0 0 0" rpy="1.5708 0 0"/>
             <geometry>
-                <cylinder radius="0.0425" length="0.110"/>
-            </geometry>
-        </collision>
-        <inertial>
-            <!-- mass=2 kg, solid cylinder r=0.0425 m, l=0.110 m -->
+               <cylinder radius="0.0425" length="0.110"/>
+            </geometry>
+        </collision>
+        <inertial>
             <origin xyz="0 0 0" rpy="0 0 0"/>
             <mass value="2.0"/>
