Commit message: delete controller

File: src/bopt_description/urdf/robot.urdf.xacro (robot description, xacro)
@@ -405,66 +405,4 @@
          FRONT WHEELS
          ================================================================ -->
-    <!-- Front socket - left (Prismatic movement) -->
-    <link name="front_socket_left">
-        <visual>
-            <origin xyz="0 0 0" rpy="0 0 0"/>
-            <geometry>
-                <mesh filename="file:///home/jkw/bopt_ws/install/bopt_description/share/bopt_description/meshes/visual/front_socket.stl"/>
-            </geometry>
-            <material name="gray"/>
-        </visual>
-        <collision>
-            <origin xyz="0 0 0" rpy="0 0 0"/>
-            <geometry>
-                <mesh filename="file:///home/jkw/bopt_ws/install/bopt_description/share/bopt_description/meshes/visual/front_socket.stl"/>
-            </geometry>
-        </collision>
-        <inertial>
-            <origin xyz="0 0 0" rpy="0 0 0"/>
-            <mass value="0.1"/>
-            <inertia ixx="0.001" ixy="0.0" ixz="0.0"
-                     iyy="0.001" iyz="0.0"
-                     izz="0.001"/>
-        </inertial>
-    </link>
-    <joint name="front_socket_left_joint" type="prismatic">
-        <parent link="front_lift_link"/>
-        <child link="front_socket_left"/>
-        <origin xyz="0.876075 0.2565 0.0176" rpy="0 0 0"/>
-        <axis xyz="1 0 0"/>
-        <limit lower="0" upper="0.00868" effort="50" velocity="2"/>
-        <dynamics damping="5.0" friction="2"/>
-    </joint>
-    <!-- Front socket - right (Prismatic movement) -->
-    <link name="front_socket_right">
-        <visual>
-            <origin xyz="0 0 0" rpy="0 0 0"/>
-            <geometry>
-                <mesh filename="file:///home/jkw/bopt_ws/install/bopt_description/share/bopt_description/meshes/visual/front_socket.stl"/>
-            </geometry>
-            <material name="gray"/>
-        </visual>
-        <collision>
-            <origin xyz="0 0 0" rpy="0 0 0"/>
-            <geometry>
-                <mesh filename="file:///home/jkw/bopt_ws/install/bopt_description/share/bopt_description/meshes/visual/front_socket.stl"/>
-            </geometry>
-        </collision>
-        <inertial>
-            <origin xyz="0 0 0" rpy="0 0 0"/>
-            <mass value="0.1"/>
-            <inertia ixx="0.001" ixy="0.0" ixz="0.0"
-                     iyy="0.001" iyz="0.0"
-                     izz="0.001"/>
-        </inertial>
-    </link>
-    <joint name="front_socket_right_joint" type="prismatic">
-        <parent link="front_lift_link"/>
-        <child link="front_socket_right"/>
-        <origin xyz="0.87605 -0.1085 0.0176" rpy="0 0 0"/>
-        <axis xyz="1 0 0"/>
-        <limit lower="0" upper="0.00868" effort="50" velocity="2"/>
-        <dynamics damping="5.0" friction="2"/>
-    </joint>
     <!-- Front wheel shaft - left -->
     <link name="front_wheel_shaft_left">
@@ -491,10 +429,18 @@
     </link>
     <joint name="front_wheel_shaft_left_joint" type="revolute">
-        <parent link="front_socket_left"/>
+        <parent link="front_lift_link"/>
         <child link="front_wheel_shaft_left"/>
-        <origin xyz="0.045125 -0.008 0" rpy="0 0.259 0"/>
+        <origin xyz="0.876075 0.2565 0.0176"
+            rpy="0 0.259 0"/>
         <axis xyz="0 1 0"/>
-        <limit lower="0" upper="0.785" effort="50" velocity="2"/>
-        <dynamics damping="5.0" friction="0.1"/>
+        <limit lower="0"
+            upper="0.73391095"
+            effort="50"
+            velocity="2"/>
+        <dynamics damping="5.0"
+                friction="0.1"/>
+        <mimic joint="front_lift_joint"
+               multiplier="7,725"
+               offset="0"/>
     </joint>
     <!-- Front wheel shaft - right -->
@@ -522,10 +468,18 @@
     </link>
     <joint name="front_wheel_shaft_right_joint" type="revolute">
-        <parent link="front_socket_right"/>
+        <parent link="front_lift_link"/>
         <child link="front_wheel_shaft_right"/>
-        <origin xyz="0.045125 -0.008 0" rpy="0 0.259 0"/>
+        <origin xyz="0.87605 -0.1085 0.0176"
+            rpy="0 0.259 0"/>
         <axis xyz="0 1 0"/>
-        <limit lower="0" upper="0.785" effort="50" velocity="2"/>
-        <dynamics damping="5.0" friction="0.1"/>
+        <limit lower="0"
+            upper="0.73391095"
+            effort="50"
+            velocity="2"/>
+        <dynamics damping="5.0"
+                friction="0.1"/>
+        <mimic joint="front_lift_joint"
+            multiplier="7.725"
+            offset="0"/>
     </joint>
     <!-- Front wheel - right -->
@@ -666,56 +620,3 @@
         <mu2>1.0</mu2>
     </gazebo>
-    <!-- ================================================================
-         ROS2 CONTROL PLUGINS AND INTERFACES
-         ================================================================ -->
-    <ros2_control name="GazeboSystem" type="system">
-        <hardware>
-            <plugin>gazebo_ros2_control/GazeboSystem</plugin>
-        </hardware>
-        <joint name="drive_wheel_Ass_joint">
-            <command_interface name="position">
-                <param name="min">-3.14159</param>
-                <param name="max">3.14159</param>
-            </command_interface>
-            <state_interface name="position"/>
-            <state_interface name="velocity"/>
-        </joint>
-        <joint name="drive_wheel_joint">
-            <command_interface name="velocity">
-                <param name="min">-3.0</param>
-                <param name="max">3.0</param>
-            </command_interface>
-            <state_interface name="position"/>
-            <state_interface name="velocity"/>
-        </joint>
-        <joint name="front_lift_joint">
-            <command_interface name="position">
-                <param name="min">0.0</param>
-                <param name="max">0.095</param>
-            </command_interface>
-            <state_interface name="position"/>
-            <state_interface name="velocity"/>
-        </joint>
-        <joint name="caster_wheel_ass_joint_left">
-            <state_interface name="position"/>
-            <state_interface name="velocity"/>
-        </joint>
-        <joint name="caster_wheel_ass_joint_right">
-            <state_interface name="position"/>
-            <state_interface name="velocity"/>
-        </joint>
-        <joint name="front_wheel_left_joint">
-            <state_interface name="position"/>
-            <state_interface name="velocity"/>
-        </joint>
-        <joint name="front_wheel_right_joint">
-            <state_interface name="position"/>
-            <state_interface name="velocity"/>
-        </joint>
-    </ros2_control>
-    <gazebo>
-        <plugin filename="libgazebo_ros2_control.so" name="gazebo_ros2_control">
-            <parameters>$(find bopt_description)/config/controllers.yaml</parameters>
-        </plugin>
-    </gazebo>
 </robot>

Commit message: create controller

File: src/bopt_description/urdf/robot.urdf.xacro (robot description, xacro)
@@ -2,4 +2,5 @@
 <robot xmlns:xacro="http://www.ros.org/wiki/xacro" name="bopt_robot">
     <xacro:include filename="materials.xacro"/>
+    <xacro:include filename="ros2_control.xacro"/>
     <!-- ================================================================
          BASE LINKS
@@ -431,9 +432,9 @@
         <parent link="front_lift_link"/>
         <child link="front_wheel_shaft_left"/>
-        <origin xyz="0.876075 0.2565 0.0176"
+        <origin xyz="0.896075 0.2565 0.0176"
             rpy="0 0.259 0"/>
         <axis xyz="0 1 0"/>
         <limit lower="0"
-            upper="0.73391095"
+            upper="0.785"
             effort="50"
             velocity="2"/>
@@ -441,5 +442,5 @@
                 friction="0.1"/>
         <mimic joint="front_lift_joint"
-               multiplier="7,725"
+               multiplier="7.725"
                offset="0"/>
     </joint>
@@ -470,9 +471,9 @@
         <parent link="front_lift_link"/>
         <child link="front_wheel_shaft_right"/>
-        <origin xyz="0.87605 -0.1085 0.0176"
+        <origin xyz="0.89605 -0.1085 0.0176"
             rpy="0 0.259 0"/>
         <axis xyz="0 1 0"/>
         <limit lower="0"
-            upper="0.73391095"
+            upper="0.785"
             effort="50"
             velocity="2"/>
@@ -543,4 +544,5 @@
         <dynamics damping="5" friction="0.1"/>
     </joint>
+    <xacro:ros2_control/>
     <!-- ================================================================
          GAZEBO MATERIALS
@@ -620,3 +622,12 @@
         <mu2>1.0</mu2>
     </gazebo>
+    <!--ROS2 Control Plugin-->
+    <gazebo>
+        <plugin name="gazebo_ros2_control"
+            filename="libgazebo_ros2_control.so">
+            <robot_param>robot_description</robot_param>
+            <robot_param_node>robot_state_publisher</robot_param_node>
+            <parameters>$(find bopt_description)/config/controller.yaml</parameters>
+        </plugin>
+    </gazebo>
 </robot>

Commit message: update thing

File: src/bopt_description/urdf/robot.urdf.xacro (robot description, xacro)
@@ -86,5 +86,5 @@
         <inertial>
             <origin xyz="0 0 0" rpy="0 0 0"/>
-            <mass value="2.0"/>
+            <mass value="3.0"/>
             <inertia ixx="0.02" ixy="0.0" ixz="0.0"
                      iyy="0.02" iyz="0.0"

File: src/bopt_description/urdf/ros2_control.xacro (robot description, xacro)
@@ -50,4 +50,20 @@
                 <state_interface name="velocity"/>
             </joint>
+            <joint name="front_wheel_shaft_left_joint">
+                <command_interface name="position">
+                    <param name="min">0.0</param>
+                    <param name="max">0.785</param>
+                </command_interface>
+                <state_interface name="position"/>
+                <state_interface name="velocity"/>
+            </joint>
+            <joint name="front_wheel_shaft_right_joint">
+                <command_interface name="position">
+                    <param name="min">0.0</param>
+                    <param name="max">0.785</param>
+                </command_interface>
+                <state_interface name="position"/>
+                <state_interface name="velocity"/>
+            </joint>
             <joint name="front_wheel_right_joint">
                 <state_interface name="position"/>

Commit message: update control

File: src/bopt_description/urdf/robot.urdf.xacro (robot description, xacro)
@@ -400,6 +400,6 @@
         <origin xyz="0.477 0 -0.265" rpy="0 0 0"/>
         <axis xyz="0 0 1"/>
-        <limit lower="0" upper="0.095" effort="30000" velocity="0.03"/>
-        <dynamics damping="50" friction="10"/>
+        <limit lower="0" upper="0.095" effort="3000" velocity="0.03"/>
+        <dynamics damping="50" friction="20"/>
     </joint>
     <!-- ================================================================
@@ -432,5 +432,5 @@
         <parent link="front_lift_link"/>
         <child link="front_wheel_shaft_left"/>
-        <origin xyz="0.896075 0.2565 0.0176"
+        <origin xyz="0.896075 0.2565 0.0196"
             rpy="0 0.259 0"/>
         <axis xyz="0 1 0"/>
@@ -471,5 +471,5 @@
         <parent link="front_lift_link"/>
         <child link="front_wheel_shaft_right"/>
-        <origin xyz="0.89605 -0.1085 0.0176"
+        <origin xyz="0.89605 -0.1085 0.0196"
             rpy="0 0.259 0"/>
         <axis xyz="0 1 0"/>

File: src/bopt_description/urdf/ros2_control.xacro (robot description, xacro)
@@ -23,7 +23,7 @@
             </joint>
             <joint name="front_lift_joint">
-                <command_interface name="effort">
-                    <param name="min">-30000</param>
-                    <param name="max">30000</param>
+                <command_interface name="position">
+                    <param name="min">0.0</param>
+                    <param name="max">0.095</param>
                 </command_interface>
                 <state_interface name="position"/>

Commit message: controller

File: src/bopt_description/urdf/robot.urdf.xacro (robot description, xacro)
@@ -24,5 +24,5 @@
         <inertial>
             <origin xyz="0 0 -0.2500" rpy="0 0 0"/>
-            <mass value="50.0"/>
+            <mass value="20.0"/>
             <inertia ixx="0.01" ixy="0.0" ixz="0.0"
                      iyy="0.01" iyz="0.0"
@@ -33,5 +33,5 @@
         <parent link="base_footprint"/>
         <child link="base_link"/>
-        <origin xyz="0 0 0.300" rpy="0 0 0"/>
+        <origin xyz="0 0 0.338" rpy="0 0 0"/>
     </joint>
     <!-- ================================================================
@@ -400,6 +400,6 @@
         <origin xyz="0.477 0 -0.265" rpy="0 0 0"/>
         <axis xyz="0 0 1"/>
-        <limit lower="0" upper="0.095" effort="3000" velocity="0.03"/>
-        <dynamics damping="50" friction="20"/>
+        <limit lower="0" upper="0.095" effort="3000" velocity="0.05"/>
+        <dynamics damping="50" friction="10"/>
     </joint>
     <!-- ================================================================

Commit message: update the controller

File: src/bopt_description/urdf/robot.urdf.xacro (robot description, xacro)
@@ -130,5 +130,5 @@
         <origin xyz="0 -0.255 -0.20515" rpy="0 0 0"/>
         <axis xyz="0 0 1"/>
-        <dynamics damping="5" friction="0.1"/>
+        <dynamics damping="1" friction="0.1"/>
     </joint>
     <!-- Caster assembly - left -->
@@ -160,5 +160,5 @@
         <origin xyz="0 0.255 -0.20515" rpy="0 0 0"/>
         <axis xyz="0 0 1"/>
-        <dynamics damping="5" friction="0.1"/>
+        <dynamics damping="1" friction="0.1"/>
     </joint>
     <!-- Caster wheel - right -->
@@ -190,5 +190,5 @@
         <origin xyz="0 0 -0.0827" rpy="0 0 0"/>
         <axis xyz="0 1 0"/>
-        <dynamics damping="5" friction="0.1"/>
+        <dynamics damping="1" friction="0.1"/>
     </joint>
     <!-- Caster wheel - left -->
@@ -220,5 +220,5 @@
         <origin xyz="0 0 -0.0827" rpy="0 0 0"/>
         <axis xyz="0 1 0"/>
-        <dynamics damping="5" friction="0.1"/>
+        <dynamics damping="1" friction="0.1"/>
     </joint>
     <!-- ================================================================
@@ -439,5 +439,5 @@
             effort="50"
             velocity="2"/>
-        <dynamics damping="5.0"
+        <dynamics damping="1.0"
                 friction="0.1"/>
         <mimic joint="front_lift_joint"
@@ -478,5 +478,5 @@
             effort="50"
             velocity="2"/>
-        <dynamics damping="5.0"
+        <dynamics damping="1.0"
                 friction="0.1"/>
         <mimic joint="front_lift_joint"
@@ -512,5 +512,5 @@
         <origin xyz="0.1488 -0.067 -0.0025435" rpy="0 -0.259 0"/>
         <axis xyz="0 1 0"/>
-        <dynamics damping="5" friction="0.1"/>
+        <dynamics damping="1" friction="0.1"/>
     </joint>
     <!-- Front wheel - left -->
@@ -542,5 +542,5 @@
         <origin xyz="0.1488 -0.067 -0.0025435" rpy="0 -0.259 0"/>
         <axis xyz="0 1 0"/>
-        <dynamics damping="5" friction="0.1"/>
+        <dynamics damping="1" friction="0.1"/>
     </joint>
     <xacro:ros2_control/>
