Commit message: Upload bopt_ws workspace (excluding large model files)

File: src/bopt_description/urdf/robot.urdf.xacro (robot description, xacro)
@@ -24,8 +24,8 @@
         <inertial>
             <origin xyz="0 0 -0.2500" rpy="0 0 0"/>
-            <mass value="20.0"/>
-            <inertia ixx="0.01" ixy="0.0" ixz="0.0"
-                     iyy="0.01" iyz="0.0"
-                     izz="0.01"/>
+            <mass value="80.0"/>
+            <inertia ixx="3.46" ixy="0.0" ixz="0.0"
+                     iyy="7.73" iyz="0.0"
+                     izz="9.06"/>
         </inertial>
     </link>
@@ -33,5 +33,5 @@
         <parent link="base_footprint"/>
         <child link="base_link"/>
-        <origin xyz="0 0 0.338" rpy="0 0 0"/>
+        <origin xyz="-1.542 0 0.337" rpy="0 0 0"/>
     </joint>
     <!-- ================================================================
@@ -55,5 +55,5 @@
         <inertial>
             <origin xyz="0 0 0" rpy="0 0 0"/>
-            <mass value="2.0"/>
+            <mass value="5.0"/>
             <inertia ixx="0.01" ixy="0.0" ixz="0.0"
                      iyy="0.01" iyz="0.0"
@@ -67,5 +67,5 @@
         <axis xyz="0 0 1"/>
         <limit lower="-3.14159" upper="3.14159" effort="1000" velocity="2"/>
-        <dynamics damping="5" friction="0.1"/>
+        <dynamics damping="6" friction="0.1"/>
     </joint>
     <!-- Drive wheel -->
@@ -83,8 +83,16 @@
                 <cylinder radius="0.115" length="0.074"/>
             </geometry>
-        </collision>
-        <inertial>
-            <origin xyz="0 0 0" rpy="0 0 0"/>
-            <mass value="3.0"/>
+            <surface>
+                <friction>
+                    <ode>
+                        <mu>1.0</mu>
+                        <mu2>1.0</mu2>
+                    </ode>
+                </friction>
+            </surface>
+        </collision>
+        <inertial>
+            <origin xyz="0 0 0" rpy="0 0 0"/>
+            <mass value="10.0"/>
             <inertia ixx="0.02" ixy="0.0" ixz="0.0"
                      iyy="0.02" iyz="0.0"
@@ -95,7 +103,7 @@
         <parent link="drive_wheel_Ass"/>
         <child link="drive_wheel"/>
-        <origin xyz="0 0 -0.223" rpy="0 0 0"/>
+        <origin xyz="0 0 -0.22315" rpy="0 0 0"/>
         <axis xyz="0 1 0"/>
-        <dynamics damping="5" friction="0.2"/>
+        <dynamics damping="10" friction="6"/>
     </joint>
     <!-- ================================================================
@@ -119,5 +127,5 @@
         <inertial>
             <origin xyz="0 0 0" rpy="0 0 0"/>
-            <mass value="1.0"/>
+            <mass value="2.0"/>
             <inertia ixx="0.02" ixy="0.0" ixz="0.0"
                      iyy="0.02" iyz="0.0"
@@ -128,7 +136,7 @@
         <parent link="base_link"/>
         <child link="caster_wheel_ass_right"/>
-        <origin xyz="0 -0.255 -0.20515" rpy="0 0 0"/>
+        <origin xyz="0 -0.255 -0.20524" rpy="0 0 0"/>
         <axis xyz="0 0 1"/>
-        <dynamics damping="1" friction="0.1"/>
+        <dynamics damping="1" friction="0.01"/>
     </joint>
     <!-- Caster assembly - left -->
@@ -149,5 +157,5 @@
         <inertial>
             <origin xyz="0 0 0" rpy="0 0 0"/>
-            <mass value="1.0"/>
+            <mass value="2.0"/>
             <inertia ixx="0.02" ixy="0.0" ixz="0.0"
                      iyy="0.02" iyz="0.0"
@@ -158,7 +166,7 @@
         <parent link="base_link"/>
         <child link="caster_wheel_ass_left"/>
-        <origin xyz="0 0.255 -0.20515" rpy="0 0 0"/>
+        <origin xyz="0 0.255 -0.20524" rpy="0 0 0"/>
         <axis xyz="0 0 1"/>
-        <dynamics damping="1" friction="0.1"/>
+        <dynamics damping="1" friction="0.01"/>
     </joint>
     <!-- Caster wheel - right -->
@@ -174,10 +182,10 @@
             <origin xyz="0 0 0" rpy="1.5708 0 0"/>
             <geometry>
-                <cylinder radius="0.050" length="0.060"/>
-            </geometry>
-        </collision>
-        <inertial>
-            <origin xyz="0 0 0" rpy="0 0 0"/>
-            <mass value="0.5"/>
+                <cylinder radius="0.050" length="0.055"/>
+            </geometry>
+        </collision>
+        <inertial>
+            <origin xyz="0 0 0" rpy="0 0 0"/>
+            <mass value="1.8"/>
             <inertia ixx="0.02" ixy="0.0" ixz="0.0"
                      iyy="0.02" iyz="0.0"
@@ -188,7 +196,7 @@
         <parent link="caster_wheel_ass_right"/>
         <child link="caster_wheel_right"/>
-        <origin xyz="0 0 -0.0827" rpy="0 0 0"/>
+        <origin xyz="0 0 -0.082835" rpy="0 0 0"/>
         <axis xyz="0 1 0"/>
-        <dynamics damping="1" friction="0.1"/>
+        <dynamics damping="10" friction="6"/>
     </joint>
     <!-- Caster wheel - left -->
@@ -204,10 +212,10 @@
             <origin xyz="0 0 0" rpy="1.5708 0 0"/>
             <geometry>
-                <cylinder radius="0.050" length="0.060"/>
-            </geometry>
-        </collision>
-        <inertial>
-            <origin xyz="0 0 0" rpy="0 0 0"/>
-            <mass value="0.5"/>
+                <cylinder radius="0.050" length="0.055"/>
+            </geometry>
+        </collision>
+        <inertial>
+            <origin xyz="0 0 0" rpy="0 0 0"/>
+            <mass value="1.8"/>
             <inertia ixx="0.02" ixy="0.0" ixz="0.0"
                      iyy="0.02" iyz="0.0"
@@ -218,7 +226,7 @@
         <parent link="caster_wheel_ass_left"/>
         <child link="caster_wheel_left"/>
-        <origin xyz="0 0 -0.0827" rpy="0 0 0"/>
+        <origin xyz="0 0 -0.082835" rpy="0 0 0"/>
         <axis xyz="0 1 0"/>
-        <dynamics damping="1" friction="0.1"/>
+        <dynamics damping="10" friction="6"/>
     </joint>
     <!-- ================================================================
@@ -388,9 +396,9 @@
         </collision>
         <inertial>
-            <origin xyz="0.477 0 0" rpy="0 0 0"/>
-            <mass value="15"/>
-            <inertia ixx="0.02" ixy="0.0" ixz="0.0"
-                     iyy="0.02" iyz="0.0"
-                     izz="0.02"/>
+            <origin xyz="0.177 0 0" rpy="0 0 0"/>
+            <mass value="25"/>
+            <inertia ixx="1.0" ixy="0.0" ixz="0.0"
+                     iyy="2.0" iyz="0.0"
+                     izz="2.0"/>
         </inertial>
     </link>
@@ -415,10 +423,10 @@
             <material name="gray"/>
         </visual>
-        <collision>
+        <!-- <collision>
             <origin xyz="0 0 0" rpy="1.5708 0 0"/>
             <geometry>
                 <mesh filename="file:///home/jkw/bopt_ws/install/bopt_description/share/bopt_description/meshes/visual/front_wheel_shaft.stl"/>
             </geometry>
-        </collision>
+        </collision> -->
         <inertial>
             <origin xyz="0.148 0 0" rpy="0 0 0"/>
@@ -432,5 +440,5 @@
         <parent link="front_lift_link"/>
         <child link="front_wheel_shaft_left"/>
-        <origin xyz="0.896075 0.2565 0.0196"
+        <origin xyz="0.9190 0.2485 0.0196"
             rpy="0 0.259 0"/>
         <axis xyz="0 1 0"/>
@@ -454,10 +462,10 @@
             <material name="gray"/>
         </visual>
-        <collision>
+        <!-- <collision>
             <origin xyz="0 0 0" rpy="1.5708 0 0"/>
             <geometry>
                 <mesh filename="file:///home/jkw/bopt_ws/install/bopt_description/share/bopt_description/meshes/visual/front_wheel_shaft.stl"/>
             </geometry>
-        </collision>
+        </collision> -->
         <inertial>
             <origin xyz="0.148 0 0" rpy="0 0 0"/>
@@ -471,5 +479,5 @@
         <parent link="front_lift_link"/>
         <child link="front_wheel_shaft_right"/>
-        <origin xyz="0.89605 -0.1085 0.0196"
+        <origin xyz="0.9190 -0.1205 0.0196"
             rpy="0 0.259 0"/>
         <axis xyz="0 1 0"/>
@@ -501,5 +509,5 @@
         <inertial>
             <origin xyz="0 0 0" rpy="0 0 0"/>
-            <mass value="2.0"/>
+            <mass value="5.0"/>
             <inertia ixx="0.01" ixy="0.0" ixz="0.0"
                      iyy="0.01" iyz="0.0"
@@ -512,5 +520,5 @@
         <origin xyz="0.1488 -0.067 -0.0025435" rpy="0 -0.259 0"/>
         <axis xyz="0 1 0"/>
-        <dynamics damping="1" friction="0.1"/>
+        <dynamics damping="10" friction="6"/>
     </joint>
     <!-- Front wheel - left -->
@@ -531,5 +539,5 @@
         <inertial>
             <origin xyz="0 0 0" rpy="0 0 0"/>
-            <mass value="2.0"/>
+            <mass value="5.0"/>
             <inertia ixx="0.01" ixy="0.0" ixz="0.0"
                      iyy="0.01" iyz="0.0"
@@ -542,5 +550,5 @@
         <origin xyz="0.1488 -0.067 -0.0025435" rpy="0 -0.259 0"/>
         <axis xyz="0 1 0"/>
-        <dynamics damping="1" friction="0.1"/>
+        <dynamics damping="10" friction="6"/>
     </joint>
     <xacro:ros2_control/>
@@ -603,14 +611,14 @@
          ================================================================ -->
     <gazebo reference="drive_wheel">
-        <mu1>1.5</mu1>
-        <mu2>1.5</mu2>
+        <mu1>2.0</mu1>
+        <mu2>2.0</mu2>
     </gazebo>
     <gazebo reference="caster_wheel_left">
-        <mu1>1.5</mu1>
-        <mu2>1.5</mu2>
+        <mu1>1.0</mu1>
+        <mu2>1.0</mu2>
     </gazebo>
     <gazebo reference="caster_wheel_right">
-        <mu1>1.5</mu1>
-        <mu2>1.5</mu2>
+        <mu1>1.0</mu1>
+        <mu2>1.0</mu2>
     </gazebo>
     <gazebo reference="front_wheel_left">
@@ -624,6 +632,6 @@
     <!--ROS2 Control Plugin-->
     <gazebo>
-        <plugin name="gazebo_ros2_control"
-            filename="libgazebo_ros2_control.so">
+        <plugin name="ign_ros2_control::IgnitionROS2ControlPlugin"
+            filename="ign_ros2_control-system">
             <robot_param>robot_description</robot_param>
             <robot_param_node>robot_state_publisher</robot_param_node>

File: src/bopt_description/urdf/ros2_control.xacro (robot description, xacro)
@@ -4,5 +4,5 @@
         <ros2_control name="my_robot_gazebo" type="system">
             <hardware>
-                <plugin>gazebo_ros2_control/GazeboSystem</plugin>
+                <plugin>ign_ros2_control/IgnitionSystem</plugin>
             </hardware>
             <joint name="drive_wheel_joint">
@@ -23,8 +23,5 @@
             </joint>
             <joint name="front_lift_joint">
-                <command_interface name="position">
-                    <param name="min">0.0</param>
-                    <param name="max">0.095</param>
-                </command_interface>
+                <command_interface name="effort"/>
                 <state_interface name="position"/>
                 <state_interface name="velocity"/>

Commit message: lift working

File: src/bopt_description/urdf/robot.urdf.xacro (robot description, xacro)
@@ -423,10 +423,10 @@
             <material name="gray"/>
         </visual>
-        <!-- <collision>
+        <collision>
             <origin xyz="0 0 0" rpy="1.5708 0 0"/>
             <geometry>
                 <mesh filename="file:///home/jkw/bopt_ws/install/bopt_description/share/bopt_description/meshes/visual/front_wheel_shaft.stl"/>
             </geometry>
-        </collision> -->
+        </collision>
         <inertial>
             <origin xyz="0.148 0 0" rpy="0 0 0"/>
@@ -462,10 +462,10 @@
             <material name="gray"/>
         </visual>
-        <!-- <collision>
+        <collision>
             <origin xyz="0 0 0" rpy="1.5708 0 0"/>
             <geometry>
                 <mesh filename="file:///home/jkw/bopt_ws/install/bopt_description/share/bopt_description/meshes/visual/front_wheel_shaft.stl"/>
             </geometry>
-        </collision> -->
+        </collision>
         <inertial>
             <origin xyz="0.148 0 0" rpy="0 0 0"/>

File: src/bopt_description/urdf/ros2_control.xacro (robot description, xacro)
@@ -47,21 +47,17 @@
                 <state_interface name="velocity"/>
             </joint>
+            <joint name="front_wheel_right_joint">
+                <state_interface name="position"/>
+                <state_interface name="velocity"/>
+            </joint>
             <joint name="front_wheel_shaft_left_joint">
-                <command_interface name="position">
-                    <param name="min">0.0</param>
-                    <param name="max">0.785</param>
-                </command_interface>
+                <param name="mimic">front_lift_joint</param>
+                <param name="multiplier">7.725</param>
                 <state_interface name="position"/>
                 <state_interface name="velocity"/>
             </joint>
             <joint name="front_wheel_shaft_right_joint">
-                <command_interface name="position">
-                    <param name="min">0.0</param>
-                    <param name="max">0.785</param>
-                </command_interface>
-                <state_interface name="position"/>
-                <state_interface name="velocity"/>
-            </joint>
-            <joint name="front_wheel_right_joint">
+                <param name="mimic">front_lift_joint</param>
+                <param name="multiplier">7.725</param>
                 <state_interface name="position"/>
                 <state_interface name="velocity"/>

Commit message: update things

File: src/bopt_description/urdf/robot.urdf.xacro (robot description, xacro)
@@ -3,4 +3,5 @@
     <xacro:include filename="materials.xacro"/>
     <xacro:include filename="ros2_control.xacro"/>
+    <xacro:include filename="gazebo.xacro"/>
     <!-- ================================================================
          BASE LINKS
@@ -553,131 +554,3 @@
     </joint>
     <xacro:ros2_control/>
-    <!-- ================================================================
-         GAZEBO MATERIALS
-         ================================================================ -->
-    <gazebo reference="base_link">
-        <material>Gazebo/Blue</material>
-    </gazebo>
-    <gazebo reference="drive_wheel_Ass">
-        <material>Gazebo/Yellow</material>
-    </gazebo>
-    <gazebo reference="drive_wheel">
-        <material>Gazebo/Black</material>
-    </gazebo>
-    <gazebo reference="caster_wheel_ass_right">
-        <material>Gazebo/Yellow</material>
-    </gazebo>
-    <gazebo reference="caster_wheel_ass_left">
-        <material>Gazebo/Yellow</material>
-    </gazebo>
-    <gazebo reference="caster_wheel_right">
-        <material>Gazebo/Black</material>
-    </gazebo>
-    <gazebo reference="caster_wheel_left">
-        <material>Gazebo/Black</material>
-    </gazebo>
-    <gazebo reference="LLt">
-        <material>Gazebo/Gray</material>
-    </gazebo>
-    <gazebo reference="LRt">
-        <material>Gazebo/Gray</material>
-    </gazebo>
-    <gazebo reference="toplidar_back">
-        <material>Gazebo/Gray</material>
-    </gazebo>
-    <gazebo reference="toplidar_front">
-        <material>Gazebo/Gray</material>
-    </gazebo>
-    <gazebo reference="top3dl_link">
-        <material>Gazebo/Gray</material>
-    </gazebo>
-    <gazebo reference="front_lift_link">
-        <material>Gazebo/Black</material>
-    </gazebo>
-    <gazebo reference="front_wheel_shaft_left">
-        <material>Gazebo/Black</material>
-    </gazebo>
-    <gazebo reference="front_wheel_shaft_right">
-        <material>Gazebo/Black</material>
-    </gazebo>
-    <gazebo reference="front_wheel_right">
-        <material>Gazebo/Black</material>
-    </gazebo>
-    <gazebo reference="front_wheel_left">
-        <material>Gazebo/Black</material>
-    </gazebo>
-    <!-- ================================================================
-         GAZEBO FRICTION PROPERTIES
-         ================================================================ -->
-    <gazebo reference="front_lift_joint">
-      <kp>100000</kp>
-      <kd>1000</kd>
-    </gazebo>
-    <gazebo reference="drive_wheel">
-        <mu1>1.2</mu1>
-        <mu2>1.2</mu2>
-        <kp>100000.0</kp>
-        <kd>100.0</kd>
-        <minDepth>0.001</minDepth>
-        <maxVel>0.1</maxVel>
-        <fdir1>1 0 0</fdir1>
-    </gazebo>
-    <gazebo reference="caster_wheel_left">
-        <mu1>0.8</mu1>   <!-- Forward friction -->
-        <mu2>0.02</mu2>  <!-- Sideways slip -->
-        <fdir1>1 0 0</fdir1>
-        <kp>100000.0</kp>
-        <kd>10.0</kd>
-        <minDepth>0.001</minDepth>
-        <maxVel>0.1</maxVel>
-    </gazebo>
-    <gazebo reference="caster_wheel_right">
-        <mu1>0.8</mu1>   <!-- Forward friction -->
-        <mu2>0.02</mu2>  <!-- Sideways slip -->
-        <fdir1>1 0 0</fdir1>
-        <kp>100000.0</kp>
-        <kd>10.0</kd>
-        <minDepth>0.001</minDepth>
-        <maxVel>0.1</maxVel>
-    </gazebo>
-    <gazebo reference="front_wheel_left">
-        <mu1>1.0</mu1>
-        <mu2>1.0</mu2>
-        <kp>100000.0</kp>
-        <kd>100.0</kd>
-        <minDepth>0.001</minDepth>
-        <maxVel>0.1</maxVel>
-    </gazebo>
-    <gazebo reference="front_wheel_right">
-        <mu1>1.0</mu1>
-        <mu2>1.0</mu2>
-        <kp>100000.0</kp>
-        <kd>100.0</kd>
-        <minDepth>0.001</minDepth>
-        <maxVel>0.1</maxVel>
-    </gazebo>
-    <gazebo reference="front_lift_joint">
-        <implicitSpringDamper>true</implicitSpringDamper>
-        <gravity>false</gravity>
-    </gazebo>
-    <!-- MIMIC STEERING JOINTS -->
-    <gazebo reference="front_wheel_shaft_left_joint">
-        <implicitSpringDamper>true</implicitSpringDamper>
-    </gazebo>
-    <gazebo reference="front_wheel_shaft_right_joint">
-        <implicitSpringDamper>true</implicitSpringDamper>
-    </gazebo>
-    <!-- DRIVE STEERING ASSEMBLY -->
-    <gazebo reference="drive_wheel_Ass_joint">
-        <implicitSpringDamper>true</implicitSpringDamper>
-    </gazebo>
-    <!--ROS2 Control Plugin-->
-    <gazebo>
-        <plugin name="ign_ros2_control::IgnitionROS2ControlPlugin"
-            filename="ign_ros2_control-system">
-            <robot_param>robot_description</robot_param>
-            <robot_param_node>robot_state_publisher</robot_param_node>
-            <parameters>$(find bopt_description)/config/controller.yaml</parameters>
-        </plugin>
-    </gazebo>
 </robot>

Commit message: small change in yaml

File: src/bopt_description/urdf/robot.urdf.xacro (robot description, xacro)
@@ -448,5 +448,5 @@
             effort="500000"
             velocity="1"/>
-        <dynamics damping="80.0"
+        <dynamics damping="125.0"
                 friction="0.8"/>
         <mimic joint="front_lift_joint"
@@ -487,5 +487,5 @@
             effort="500000"
             velocity="1"/>
-        <dynamics damping="80.0"
+        <dynamics damping="125.0"
                 friction="0.8"/>
         <mimic joint="front_lift_joint"

Commit message: update sensor

File: src/bopt_description/urdf/robot.urdf.xacro (robot description, xacro)
@@ -377,5 +377,5 @@
         <parent link="base_link"/>
         <child link="top3dl_link"/>
-        <origin xyz="0.2356 0.0024 1.9831" rpy="0 0 0"/>
+        <origin xyz="0.2556 0.0024 1.9831" rpy="0 0 0"/>
     </joint>
     <!-- ================================================================

Commit message: fix the height issue

File: src/bopt_description/urdf/robot.urdf.xacro (robot description, xacro)
@@ -65,5 +65,5 @@
         <parent link="base_link"/>
         <child link="drive_wheel_Ass"/>
-        <origin xyz="0 0 0" rpy="0 0 0"/>
+        <origin xyz="0 0 -0.000849" rpy="0 0 0"/>
         <axis xyz="0 0 1"/>
         <limit lower="-3.14159" upper="3.14159" effort="1000" velocity="2"/>
@@ -118,5 +118,5 @@
         <parent link="drive_wheel_Ass"/>
         <child link="drive_wheel"/>
-        <origin xyz="0 0 -0.22315" rpy="0 0 0"/>
+        <origin xyz="0 0 -0.21916" rpy="0 0 0"/>
         <axis xyz="0 1 0"/>
         <dynamics damping="10" friction="6"/>
@@ -151,5 +151,5 @@
         <parent link="base_link"/>
         <child link="caster_wheel_ass_right"/>
-        <origin xyz="0 -0.255 -0.20524" rpy="0 0 0"/>
+        <origin xyz="0 -0.26066 -0.205" rpy="0 0 0"/>
         <axis xyz="0 0 1"/>
         <dynamics damping="1" friction="0.01"/>
@@ -181,5 +181,5 @@
         <parent link="base_link"/>
         <child link="caster_wheel_ass_left"/>
-        <origin xyz="0 0.255 -0.20524" rpy="0 0 0"/>
+        <origin xyz="0 0.26066 -0.205" rpy="0 0 0"/>
         <axis xyz="0 0 1"/>
         <dynamics damping="1" friction="0.01"/>
@@ -211,5 +211,5 @@
         <parent link="caster_wheel_ass_right"/>
         <child link="caster_wheel_right"/>
-        <origin xyz="0 0 -0.082835" rpy="0 0 0"/>
+        <origin xyz="0 0 -0.080" rpy="0 0 0"/>
         <axis xyz="0 1 0"/>
         <dynamics damping="10" friction="6"/>
@@ -241,5 +241,5 @@
         <parent link="caster_wheel_ass_left"/>
         <child link="caster_wheel_left"/>
-        <origin xyz="0 0 -0.082835" rpy="0 0 0"/>
+        <origin xyz="0 0 -0.080" rpy="0 0 0"/>
         <axis xyz="0 1 0"/>
         <dynamics damping="10" friction="6"/>

Commit message: nmpc controller

File: src/bopt_description/urdf/robot.urdf.xacro (robot description, xacro)
@@ -65,5 +65,5 @@
         <parent link="base_link"/>
         <child link="drive_wheel_Ass"/>
-        <origin xyz="0 0 -0.000849" rpy="0 0 0"/>
+        <origin xyz="0 0 -0.00086" rpy="0 0 0"/>
         <axis xyz="0 0 1"/>
         <limit lower="-3.14159" upper="3.14159" effort="1000" velocity="2"/>

Commit message: update things of nmpc

File: src/bopt_description/urdf/robot.urdf.xacro (robot description, xacro)
@@ -65,5 +65,5 @@
         <parent link="base_link"/>
         <child link="drive_wheel_Ass"/>
-        <origin xyz="0 0 -0.00086" rpy="0 0 0"/>
+        <origin xyz="0 0 -0.00087" rpy="0 0 0"/>
         <axis xyz="0 0 1"/>
         <limit lower="-3.14159" upper="3.14159" effort="1000" velocity="2"/>

Commit message: multiplt robot

File: src/bopt_description/urdf/robot.urdf.xacro (robot description, xacro)
@@ -65,5 +65,5 @@
         <parent link="base_link"/>
         <child link="drive_wheel_Ass"/>
-        <origin xyz="0 0 -0.00087" rpy="0 0 0"/>
+        <origin xyz="0 0 -0.0010" rpy="0 0 0"/>
         <axis xyz="0 0 1"/>
         <limit lower="-3.14159" upper="3.14159" effort="1000" velocity="2"/>

Commit message: sdfgsd

File: src/bopt_description/urdf/robot.urdf.xacro (robot description, xacro)
@@ -85,7 +85,7 @@
     </link>
     <joint name="imu_joint" type="fixed">
-        <parent link="drive_wheel_Ass"/>
+        <parent link="base_link"/>
         <child link="imu_link"/>
-        <origin xyz="0 0 0.01"/>
+        <origin xyz="0 0 0"/>
     </joint>
     <!-- Drive wheel -->
@@ -106,6 +106,6 @@
                 <friction>
                     <ode>
-                        <mu>1.5</mu>
-                        <mu2>1.5</mu2>
+                        <mu>5.0</mu>
+                        <mu2>5.0</mu2>
                     </ode>
                 </friction>
